File: hardware/80m/01_source_interface.kicad_sch (KiCad schematic)
At the start: 23 parts, among them J101 IDC16 controller, U101 SI5351A-B-GT, Y101 25 MHz / CL10 pF

Commit message: Correct RF80 timer polarities and arming logic for M3A-R1 review
Other:
- note added: "M3A-R1: REVIEW / ALL hardware measurements NOT RUN / no layout or procurement."
- note removed: "M3A-R0: REVIEW / ALL hardware measurements NOT RUN / no layout or procurement."

Commit message: Preserve M3B-E1 evaluation PCB before independent-review corrections
Parts:
- C101, C102: Engineering_Note Dated M2 distributor observation; no fresh basket verificat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 -> (none)
- J101: footprint Connector_IDC:IDC-Header_2x08_P2.54mm_Vertical -> ARDF_TX:Wurth_61201621621; Engineering_Note Exact Wurth drawing/key orientation to verify; candidate fo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 -> Maker61201621621:27.98mm length,17.78mm span,2.54mm pitch; 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
- TP101, TP102, TP103, TP104, TP105: now left out of the parts list
- U101: Engineering_Note 0x60; CLK0 PA, CLK2 FOX; CLK1 disabled/NC; blank factory part, no preprogrammed outputs. Internal crystal load 10 pF starting setting. Dated M2 distributor observation; no fresh basket verification. -> 0x60; CLK0 PA, CLK2 FOX; CLK1 disabled/NC; blank factory part, no preprogrammed outputs. Internal crystal load 10 pF starting setting.
Other:
- note added: "M3B-E1: REVIEW / ALL hardware measurements NOT RUN / no ordering or manufacture."
- note removed: "M3A-R1: REVIEW / ALL hardware measurements NOT RUN / no layout or procurement."

Commit message: Correct RF80 M3B-E2 physical pinouts and audit manufacturing readiness
Other:
- note added: "M3B-E2: REVIEW / ALL hardware measurements NOT RUN / no ordering or manufacture."
- note removed: "M3B-E1: REVIEW / ALL hardware measurements NOT RUN / no ordering or manufacture."
