File: hardware/80m/04_arm_key.kicad_sch (KiCad schematic)
At the start: 8 parts, among them U221 74HC11D,653, U222 74HC08D,653, U223 74HC74D,653, U224 74HC74D,653

Commit message: Correct RF80 timer polarities and arming logic for M3A-R1 review
Parts:
- removed unit 3 of U224
- removed unit 2 of U224
- added Q225, Q226, Q227, Q228, Q229: BSS138BK,215, Package_TO_SOT_SMD:SOT-23, symbol ARDF_TX:2N7002
- C233: Population NORMAL -> BOTH
- U224: value 74HC74D,653 -> 74HC174D,653; footprint Package_SO:SOIC-14_3.9x8.7mm_P1.27mm -> Package_SO:SOIC-16_3.9x9.9mm_P1.27mm; symbol ARDF_TX:74HC74 -> ARDF_TX:74HC174; Engineering_Note CMOS 3.3 V. Supply unit and all unused gates explicitly connected. Dated M2 distributor observation; no fresh basket verification. -> CMOS 3.3 V. Supply unit and all unused gates explicitly connected.; MPN 74HC74D,653 -> 74HC174D,653; Population NORMAL -> BOTH
Connections:
- net SAFE12 is gone; now on net POR_N: U221.1
- net THERM_OK is gone; now on net BUS_LINES_HIGH: U222.11
- net ARM: now also U224.9 (Cp)
- net ARM_CLK: no longer U224.3 (C)
- net FOX_REQ: now also U224.11 (D3); no longer U221.10
- net FOX_REQ_N: now also Q228.1 (G); no longer U221.5
- net GND: now also U224.14 (D5), U224.8 (GND), Q229.2 (S); no longer U223.11 (C), U223.12 (D)
- net PA_REQ: now also U224.6 (D2); no longer U221.4
- net PA_REQ_N: now also Q226.1 (G); no longer U221.11
- net PWR0: now also U224.3 (D0); no longer U224.2 (D)
- net PWR1: now also U224.4 (D1)
- net SEL_EXT: now also U224.2 (Q0); no longer U224.5 (Q)
- net SEL_FULL: now also U224.5 (Q1)
- net V3V3: now also U223.12 (D), U224.16 (VCC); no longer U223.2 (D), U224.4 (~{S})
- net LEASE_SEEN_N: now reaches U223.8 (~{Q})
- net CLR_N renamed RESET_N
- net RESET_N: no longer U224.1 (~{R})
- net SAFE_MODES renamed BUS_HOLDOFF_N
- net SAFE_PACK renamed BUS_LINES_HIGH
- net SAFE_RAW renamed BUS_QUIET
- net BUS_QUIET: no longer U222.1
- net TEMP_HOT_OK renamed SCL
- net TEMP_OPEN_OK renamed SDA
- new net ARM_ACCEPT: Q229.1 (G), U221.11, U221.5, U223.2 (D), U224.12 (Q4)
- new net DROP_RETURN: Q226.2 (S), Q228.2 (S), Q229.3 (D)
- new net FOX_DROP_MID: Q227.2 (S), Q228.3 (D)
- new net HEALTH_N: Q225.3 (D), Q227.3 (D), U222.1, U224.1 (~{Mr})
- new net KEY_N: U224.13 (D4)
- new net LEASE: U223.11 (C)
- new net PATH_FOX: Q227.1 (G), U221.10, U224.10 (Q3)
- new net PATH_PA: Q225.1 (G), U221.4, U224.7 (Q2)
- new net PA_DROP_MID: Q225.2 (S), Q226.3 (D)
- no-connect marks 4 -> 2
Other:
- note added: "04 Deliberate rearm, witnessed heartbeat and captured configuration"
- note added: "M3A-R1: REVIEW / ALL hardware measurements NOT RUN / no layout or procurement."
- note added: "U224 captures path/mode/key-low on raw ARM; any health fault clears acceptance. U223 delayed clock can only arm an accepted context. A fault in the pending delay cannot rearm. Withdraw selected request: health clears context and RF permits. New raw ARM edge required. Fresh ARM low>=20ms, configure requests/mode, then ARM high; wait>=250ms before first key. Mode changes while armed are ignored; mo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"
- note removed: "04 Rearm latch, selected rails and key permits"
- note removed: "M3A-R0: REVIEW / ALL hardware measurements NOT RUN / no layout or procurement."
- note removed: "PWR1/PWR0: 00 Sprint (start4.68V); 01 extended (start5.58V); 10 full (start7.96V); 11 fault. Modes latch on delayed ARM edge and reset to Sprint on fault. Changing PWR while armed does not change rail; changing to11 still faults. Retuning/I2C, stopped heartbeat, MUTE low, UV/OV/OC/hot/open NTC clear ARMED. Rearm: ARM low >=20ms, health stable + I2C quiet, requests/mode fixed; ARM high then wait >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"
- title: 04 Rearm latch, selected rails and key permits -> 04 Deliberate rearm, witnessed heartbeat and captured configuration

Commit message: Preserve M3B-E1 evaluation PCB before independent-review corrections
Parts:
- C230, C231, C232, C233: Engineering_Note Dated M2 distributor observation; no fresh basket verificat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 -> (none)
- U222, U223: Engineering_Note CMOS 3.3 V. Supply unit and all unused gates explicitly connected. Dated M2 distributor observation; no fresh basket verification. -> CMOS 3.3 V. Supply unit and all unused gates explicitly connected.
Other:
- note added: "M3B-E1: REVIEW / ALL hardware measurements NOT RUN / no ordering or manufacture."
- note removed: "M3A-R1: REVIEW / ALL hardware measurements NOT RUN / no layout or procurement."

Commit message: Correct RF80 M3B-E2 physical pinouts and audit manufacturing readiness
Other:
- note added: "M3B-E2: REVIEW / ALL hardware measurements NOT RUN / no ordering or manufacture."
- note removed: "M3B-E1: REVIEW / ALL hardware measurements NOT RUN / no ordering or manufacture."
