File: hardware/80m/05_power.kicad_sch (KiCad schematic)
At the start: 22 parts, among them J301 RAW protected pack, Q301 DMN2056U-7, Q302 DMN2056U-7, U301 TPS54302DDCT, U302 TPS22810DBVR

Commit message: Correct RF80 timer polarities and arming logic for M3A-R1 review
Parts:
- C306: value 1n -> 4.7n; Engineering_Note Slew timing starter, measure real charge current and disabl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 -> 4.7n slows initial47uFdrivercharge; measure inrush belowOC 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; MPN CC0603JRNPO9BN102 -> CC0603JRNPO9BN472
- Q301, Q302: value DMN2056U-7 -> BSS138BK,215; Engineering_Note 20VDS, +/-8VGS;45mohm at2.5V. Native2N7002 drawing only, ac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 -> 60VDS,+/-20VGS;6.5ohm max at2.5V/10mA. Low-current function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; MPN DMN2056U-7 -> BSS138BK,215
Other:
- note added: "M3A-R1: REVIEW / ALL hardware measurements NOT RUN / no layout or procurement."
- note added: "Shared J301/F301/D301 input barrier; converter/loadswitch NORMAL only. Protected4S:12.0-16.8V. Fox-only retains input barrier/sense bypass, omits buck/loadswitch and watt-rail parts;2S powerscontroller+input sense. TPS22810 VIN must stay<=18V, including failed-buck transients;20V is absolute maximum. 28V passive simulation is NOT a system rating. Input clamp/fault coordination remains OPEN."
- note removed: "M3A-R0: REVIEW / ALL hardware measurements NOT RUN / no layout or procurement."
- note removed: "Shared J301/F301/D301 input barrier; converter/loadswitch NORMAL only. Protected4S:12.0-16.8V. Fox-only retains input barrier/sense bypass, omits buck/loadswitch and watt-rail parts;2S powerscontroller+input sense."

Commit message: Preserve M3B-E1 evaluation PCB before independent-review corrections
Parts:
- C303: Engineering_Note Dated M2 distributor observation; no fresh basket verificat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 -> (none)
- D301: Engineering_Note Schottky reverse polarity barrier; K pin1 = VIN_PA. Vf/cond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 -> Schottky reverse polarity barrier. M3B sense is ahead of ad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
- D302: Engineering_Note Nominal clamp27.6V close to28V recommended input; real cabl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 -> Secondary surge absorber only; NOT an18/20V precision clamp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
- F301: footprint Fuse:Fuse_1206_3216Metric -> ARDF_TX:Fuse_467_0603; Engineering_Note Selection candidate; final interrupt/I2t and max16.8V quali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 -> CORRECTED R1 footprint: actual467 family is0603. Own maker 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
Connections:
- net VIN_PA: no longer D301.1 (K)
- new net VIN_PACK: D301.1 (K)
Other:
- note added: "M3B-E1: REVIEW / ALL hardware measurements NOT RUN / no ordering or manufacture."
- note removed: "M3A-R1: REVIEW / ALL hardware measurements NOT RUN / no layout or procurement."

Commit message: Correct RF80 M3B-E2 physical pinouts and audit manufacturing readiness
Parts:
- D302: Engineering_Note Secondary surge absorber only; NOT an18/20V precision clamp. M3B R350/C350 damp specified cable hot-plug; TVS is downstream of damper. External sources restricted to qualified4S envelope. -> Secondary surge absorber only; NOT an18/20V precision clamp. M3B R350/C350 damp specified cable hot-plug; TVS is downstream of damper. External sources restricted to qualified4S envelope. E2 exact vendor LittelfuseSMBJ17A:17V stand-off,18.9-20.9V breakdown at1mA,27.6V clamp at21.8A. Existing EUR0.35 remains unquoted estimate; not an18V limiter.; Manufacturer (none) -> Littelfuse
Other:
- note added: "M3B-E2: REVIEW / ALL hardware measurements NOT RUN / no ordering or manufacture."
- note removed: "M3B-E1: REVIEW / ALL hardware measurements NOT RUN / no ordering or manufacture."
