File: hardware/80m/06_analog_protection.kicad_sch (KiCad schematic)
At the start: 17 parts, among them U311 TL431AIDBZR, U312 LM339BIDR

Commit message: Correct RF80 timer polarities and arming logic for M3A-R1 review
Parts:
- removed R320, R322, R323: 10k, Resistor_SMD:R_0603_1608Metric, symbol ARDF_TX:R
- C310, C313, R311, R312, R324, R325, U312: Population BOTH -> NORMAL
- R321: value 10k -> 2.2k; Engineering_Note Dated M2 distributor observation; no fresh basket verificat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 -> (none); MPN RC0603FR-0710KL -> RC0603FR-072K2L; Population BOTH -> NORMAL
Connections:
- net LOCAL_4S_OK is gone; now on net PA_GUARD_RAW: R321.2, U312.1
- net PA_OC_OK is gone; now on net PA_GUARD_RAW: U312.14
- net PA_OV_OK is gone; now on net PA_GUARD_RAW: U312.13
- net V_PACK_SCALED: no longer U312.5 (+)
- net COMMON_UV_OK renamed PA_GUARD_RAW
- net PACK_2S_REF renamed TEMP_HOT_REF
- new net TEMP_SENSE: U312.5 (+)
Other:
- note added: "M3A-R1: REVIEW / ALL hardware measurements NOT RUN / no layout or procurement."
- note added: "Nominal backup: commonUV5.810V/4Sbackup11.070V postreversebarrier; railOV8.973V. Controller operational endpoint remains6.0/12.0V with hysteresis; cell-group BMS external. Local pack sensing does not prove weakest-cell voltage. Hysteresis implemented by fault latch; rearm only after input exceeds qualified margin. Fox-only: watt guards DNP, R228 clamps PA_GUARD_RAW; UV comparator remains local."
- note removed: "M3A-R0: REVIEW / ALL hardware measurements NOT RUN / no layout or procurement."
- note removed: "Nominal backup: commonUV5.810V/4Sbackup11.070V postreversebarrier; railOV8.973V. Controller operational endpoint remains6.0/12.0V with hysteresis; cell-group BMS external. Local pack sensing does not prove weakest-cell voltage. Hysteresis implemented by fault latch; rearm only after input exceeds qualified margin. Fox-only: VPA node is grounded via R325/R324, not floating."
- moved on the sheet: R321

Commit message: Preserve M3B-E1 evaluation PCB before independent-review corrections
Parts:
- C310, C313, R314, R325: Engineering_Note Dated M2 distributor observation; no fresh basket verificat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 -> (none)
- C314: Engineering_Note Dated M2 distributor observation; no fresh basket verificat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 -> 50V version on undamped VIN_PACK node; avoids crediting the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; MPN CC0603KRX7R8BB104 -> CC0603KRX7R9BB104
Connections:
- net VIN_PA renamed VIN_PACK
Other:
- note added: "M3B-E1: REVIEW / ALL hardware measurements NOT RUN / no ordering or manufacture."
- note removed: "M3A-R1: REVIEW / ALL hardware measurements NOT RUN / no layout or procurement."

Commit message: Correct RF80 M3B-E2 physical pinouts and audit manufacturing readiness
Parts:
- U311: symbol ARDF_TX:TL431DBZ -> ARDF_TX:TL431_TI_DBZ; Engineering_Note 1 REF,2 anode,3 cathode. >=1mA reference bias; no capacitor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 -> TI TL431AIDBZR DBZ, SLVS543S May2024 Table5-1/p4:1CATHODE,2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; Manufacturer (none) -> Texas Instruments
Connections:
- net GND: now also U311.3 (A); no longer U311.2 (REF)
- net VREF_2V5: now also U311.2 (REF); no longer U311.3 (A)
Other:
- note added: "M3B-E2: REVIEW / ALL hardware measurements NOT RUN / no ordering or manufacture."
- note removed: "M3B-E1: REVIEW / ALL hardware measurements NOT RUN / no ordering or manufacture."
