File: hardware/80m/07_current_thermal.kicad_sch (KiCad schematic)
At the start: 20 parts, among them U313 INA180A1IDBVT, U314 LM393BIDR

Commit message: Correct RF80 timer polarities and arming logic for M3A-R1 review
Parts:
- removed R336, R341, R342: 10k, Resistor_SMD:R_0603_1608Metric, symbol ARDF_TX:R
- added R348, R349: 0, Resistor_SMD:R_0603_1608Metric, symbol ARDF_TX:R
- R334, R335, R337, R338, R339, R340: Population BOTH -> NORMAL
- TH301: Engineering_Note B25/50=3380K;3434K25/85referenceusedforapproximate80Ctrip,notconstantovertemperature. Manufacturerproductpageunavailable; supplier-hostedMuratasheetreviewrequired. Attach sensor thermally to IRF610 case; board0603 placement cannot substitute case sensing. Fox-only fit fixed10k instead via R336. -> B25/50=3380K;3434K25/85referenceusedforapproximate80Ctrip,notconstantovertemperature. Manufacturerproductpageunavailable; supplier-hostedMuratasheetreviewrequired. Attach sensor thermally to IRF610 case; board0603 placement cannot substitute case sensing. Fox-only DNP; normal PA and thermal sensing absent; unused dual-comparator inputs grounded via R348/R349.; Population BOTH -> NORMAL
Connections:
- net GND: now also R348.2, R349.2
- net TEMP_HOT_REF: no longer U314.2 (-)
- net TEMP_OPEN_REF: now also R348.1
- net TEMP_SENSE: now also R349.1; no longer U314.3 (+)
- net TEMP_HOT_OK renamed UV_POR_N
- net TEMP_OPEN_OK renamed PA_GUARD_RAW
- new net PACK_2S_REF: U314.2 (-)
- new net V_PACK_SCALED: U314.3 (+)
Other:
- note added: "M3A-R1: REVIEW / ALL hardware measurements NOT RUN / no layout or procurement."
- note removed: "M3A-R0: REVIEW / ALL hardware measurements NOT RUN / no layout or procurement."

Commit message: Preserve M3B-E1 evaluation PCB before independent-review corrections
Parts:
- C322, C323, R338, R340, U314: Engineering_Note Dated M2 distributor observation; no fresh basket verificat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 -> (none)
- R334: Engineering_Note Shared default0V OC input with sensor DNP; valid only when watt stage DNP. Dated M2 distributor observation; no fresh basket verification. -> Shared default0V OC input with sensor DNP; valid only when watt stage DNP.
- R335: Engineering_Note Pull from bounded<1.0V reference keeps comparator inputs in range at cold/open NTC. Dated M2 distributor observation; no fresh basket verification. -> Pull from bounded<1.0V reference keeps comparator inputs in range at cold/open NTC.
- R348, R349: now not fitted
- U313: Engineering_Note Gain20V/V; pin3 IN+,4 IN-,5 VS for DBV. 26V CM. A1T packaging differs from unavailable A1R, same pinout. Quantity10EUR0.70 isESTIMATE; EUR0.96 at1 observed. -> Gain20V/V; pin3 IN+,4 IN-,5 VS for DBV. 26V CM. A1T packaging differs from unavailable A1R, same pinout.
Other:
- note added: "M3B-E1: REVIEW / ALL hardware measurements NOT RUN / no ordering or manufacture."
- note removed: "M3A-R1: REVIEW / ALL hardware measurements NOT RUN / no layout or procurement."

Commit message: Correct RF80 M3B-E2 physical pinouts and audit manufacturing readiness
Other:
- note added: "M3B-E2: REVIEW / ALL hardware measurements NOT RUN / no ordering or manufacture."
- note removed: "M3B-E1: REVIEW / ALL hardware measurements NOT RUN / no ordering or manufacture."
