File: hardware/80m/09_normal_filter.kicad_sch (KiCad schematic)
At the start: 15 parts, among them J401 NORMAL 50ohm reference

Commit message: Correct RF80 timer polarities and arming logic for M3A-R1 review
Other:
- note added: "M3A-R1: REVIEW / ALL hardware measurements NOT RUN / no layout or procurement."
- note removed: "M3A-R0: REVIEW / ALL hardware measurements NOT RUN / no layout or procurement."

Commit message: Preserve M3B-E1 evaluation PCB before independent-review corrections
Parts:
- TP410, TP411, TP412, TP413, TP414: now left out of the parts list
Other:
- note added: "M3B-E1: REVIEW / ALL hardware measurements NOT RUN / no ordering or manufacture."
- note removed: "M3A-R1: REVIEW / ALL hardware measurements NOT RUN / no layout or procurement."

Commit message: Correct RF80 M3B-E2 physical pinouts and audit manufacturing readiness
Other:
- note added: "M3B-E2: REVIEW / ALL hardware measurements NOT RUN / no ordering or manufacture."
- note removed: "M3B-E1: REVIEW / ALL hardware measurements NOT RUN / no ordering or manufacture."
