File: hardware/80m/10_fox_rf.kicad_sch (KiCad schematic)
At the start: 19 parts, among them Q501 MMBT3906,215, Q502 DMN2056U-7, Q503 MMBT3904,215, Q504 MMBT3904,215, U501 SN74AC00DR

Commit message: Correct RF80 timer polarities and arming logic for M3A-R1 review
Parts:
- Q502: value DMN2056U-7 -> BSS138BK,215; Engineering_Note 20VDS, +/-8VGS;45mohm at2.5V. Native2N7002 drawing only, ac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 -> 60VDS,+/-20VGS;6.5ohm max at2.5V/10mA. Low-current function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; MPN DMN2056U-7 -> BSS138BK,215
Other:
- note added: "M3A-R1: REVIEW / ALL hardware measurements NOT RUN / no layout or procurement."
- note removed: "M3A-R0: REVIEW / ALL hardware measurements NOT RUN / no layout or procurement."

Commit message: Preserve M3B-E1 evaluation PCB before independent-review corrections
Parts:
- C502, R505, R508, R509: Engineering_Note Dated M2 distributor observation; no fresh basket verificat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 -> (none)
- TP501, TP502: now left out of the parts list
Other:
- note added: "M3B-E1: REVIEW / ALL hardware measurements NOT RUN / no ordering or manufacture."
- note removed: "M3A-R1: REVIEW / ALL hardware measurements NOT RUN / no layout or procurement."

Commit message: Correct RF80 M3B-E2 physical pinouts and audit manufacturing readiness
Other:
- note added: "M3B-E2: REVIEW / ALL hardware measurements NOT RUN / no ordering or manufacture."
- note removed: "M3B-E1: REVIEW / ALL hardware measurements NOT RUN / no ordering or manufacture."
