File: hardware/80m/12_evaluation.kicad_sch (KiCad schematic)
At the start: 55 parts

Commit message: Correct RF80 M3B-E2 physical pinouts and audit manufacturing readiness
Other:
- note added: "M3B-E2: REVIEW / ALL hardware measurements NOT RUN / no ordering or manufacture."
- note added: "M3B-E2: bounded12.0-16.8V protected4S only; first bring-up uses a CURRENT-LIMITED LAB SUPPLY. R350/C350 damp cable L<=10uH; pack sense remains ahead of R350. TVS is NOT an18V clamp. No driver fitted until power-only OV withdrawal test proves VDRV<=12.6V. No physical tests performed."
- note removed: "M3B-E1: REVIEW / ALL hardware measurements NOT RUN / no ordering or manufacture."
- note removed: "M3B-E1: bounded12.0-16.8V protected4S only; first bring-up uses a CURRENT-LIMITED LAB SUPPLY. R350/C350 damp cable L<=10uH; pack sense remains ahead of R350. TVS is NOT an18V clamp. No driver fitted until power-only OV withdrawal test proves VDRV<=12.6V. No physical tests performed."
