File: hardware/80m/RF80.kicad_pcb (KiCad board)
At the start: 2 copper layers, 210 x 160 mm, 277 parts, among them J101 IDC16 controller, J301 RAW protected pack, J401 NORMAL 50ohm reference, J502 FOX ONLY / compact, Q201 BSS138BK,215, Q225 BSS138BK,215, Q226 BSS138BK,215, Q227 BSS138BK,215, Q228 BSS138BK,215, Q229 BSS138BK,215, Q301 BSS138BK,215, Q302 BSS138BK,215, Q401 BSS138BK,215, Q402 IRF610PBF-BE3, Q403 BD140 / ST, Q404 DMN2056U-7, Q405 BSS138BK,215, Q406 BSS138BK,215, Q501 MMBT3906,215, Q502 BSS138BK,215, Q503 MMBT3904,215, Q504 MMBT3904,215, T401 9T + 9T bifilar / FT-50A-43, U101 SI5351A-B-GT, U201 MCP100T-300I/TT, U202 74HC123D,653, U203 74HC14D,653, U211 74HC21D,653, U212 74HC00D,653, U221 74HC11D,653, U222 74HC08D,653, U223 74HC74D,653, U224 74HC174D,653, U301 TPS54302DDCT, U302 TPS22810DBVR, U311 TL431AIDBZR, U312 LM339BIDR, U313 INA180A1IDBVT, U314 LM393BIDR, U401 LM5134BMF/NOPB, U501 SN74AC00DR, Y101 25 MHz / CL10 pF

Commit message: Correct RF80 M3B-E2 physical pinouts and audit manufacturing readiness
Parts:
- Q403: footprint Package_TO_SOT_THT:TO-126-3_Vertical -> ARDF_TX:ST_BD140_SOT32_1p3Drill
- moved Q403 4.56 mm to (160.6, 69.0), turned to 180 degrees
Connections:
- Q403 pad 1: VPA_LOAD -> SHAPE_BASE
- Q403 pad 3: SHAPE_BASE -> VPA_LOAD
- U311 pad 2: GND -> VREF_2V5
- U311 pad 3: VREF_2V5 -> GND
Routing:
- net GND: vias 129 -> 130
Other:
- rule pad_to_mask_clearance: 0 -> 0.025
- board text added: "3:E 2:C 1:B"
- board text added: "ARDF-TX RF80 / M3B-E2 EVALUATION"
- board text added: "ST BD140: DRAWING FACE TOWARD +Y"
- board text removed: "ARDF-TX RF80 / M3B-E1 EVALUATION"
Changed lines of the file:
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@@
 	(title_block
 		(title "RF80 80 m evaluation PCB - ENGINEERING REVIEW")
-		(date "2026-10-14")
-		(rev "M3B-E1")
+		(date "2026-10-15")
+		(rev "M3B-E2")
 		(company "ARDF-TX")
 		(comment 1 "UNBUILT - NOT A MANUFACTURING RELEASE")
@@
 	)
 	(setup
-		(pad_to_mask_clearance 0)
+		(pad_to_mask_clearance 0.025)
+		(solder_mask_min_width 0.075)
 		(allow_soldermask_bridges_in_footprints no)
 		(tenting
@@
 			)
 		)
-		(property "Datasheet" ""
+		(property "Datasheet" "https://www.littelfuse.com/assetdocs/littelfuse_tvs_diode_smbj_datasheet.pdf?assetguid=09a6ae9a-73cb-4ac4-acac-e6dab92ab953"
 			(at 0 0 90)
 			(unlocked yes)
@@
 			)
 		)
-		(property "Engineering_Note" "Secondary surge absorber only; NOT an18/20V precision clamp. M3B R350/C350 damp specified cable hot-plug; TVS is downstream of damper. External sources restricted to qualified4S envelope."
+		(property "Engineering_Note" "Secondary surge absorber only; NOT an18/20V precision clamp. M3B R350/C350 damp specified cable hot-plug; TVS is downstream of damper. External sources restricted to qualified4S envelope. E2 exact vendor LittelfuseSMBJ17A:17V stand-off,18.9-20.9V breakdown at1mA,27.6V clamp at21.8A. Existing EUR0.35 remains unquoted estimate; not an18V limiter."
 			(at 0 0 90)
 			(layer "F.SilkS")
@@
 			)
 		)
+		(property "Manufacturer" "Littelfuse"
+			(at 0 0 0)
+			(layer "F.SilkS")
+			(hide yes)
+			(effects
+				(font
+					(size 1.27 1.27)
+					(thickness 0.15)
+				)
+			)
+		)
 		(attr smd)
 		(duplicate_pad_numbers_are_jumpers no)
@@
 		)
 	)
-	(footprint "Package_TO_SOT_THT:TO-126-3_Vertical"
+	(footprint "ARDF_TX:ST_BD140_SOT32_1p3Drill"
 		(layer "F.Cu")
-		(at 156 69)
+		(at 160.56 69 180)
 		(descr "TO-126-3, Vertical, RM 2.28mm, see https://www.diodes.com/assets/Package-Files/TO126.pdf")
 		(tags "TO-126-3 Vertical RM 2.28mm")
 		(property "Reference" "Q403"
-			(at 2.28 -2.95 0)
+			(at 2.28 -2.95 180)
 			(layer "F.Fab")
 			(effects
@@
 		)
 		(property "Value" "BD140 / ST"
-			(at 2.28 2.2 0)
+			(at 2.28 2.2 180)
 			(layer "F.Fab")
 			(hide yes)
@@
 		)
 		(property "Datasheet" "https://www.st.com/resource/en/datasheet/bd140.pdf"
-			(at 0 0 0)
+			(at 0 0 180)
 			(layer "F.Fab")
 			(hide yes)
@@
 		)
 		(property "Description" ""
-			(at 0 0 0)
+			(at 0 0 180)
 			(layer "F.Fab")
 			(hide yes)
@@
 		)
 		(property "KiLib_Generator" "package/TO_SOT/THT"
-			(at 0 0 0)
+			(at 0 0 180)
 			(layer "F.SilkS")
 			(hide yes)
@@
 		)
 		(property "MPN" "BD140"
-			(at 0 0 0)
+			(at 0 0 180)
 			(layer "F.SilkS")
 			(hide yes)
@@
 		)
 		(property "Population" "NORMAL"
-			(at 0 0 0)
+			(at 0 0 180)
 			(layer "F.SilkS")
 			(hide yes)
@@
 		)
 		(property "Function" "normal_shaper"
-			(at 0 0 0)
+			(at 0 0 180)
+			(layer "F.SilkS")
+			(hide yes)
+			(effects
+				(font
+					(size 1.27 1.27)
+					(thickness 0.15)
+				)
+			)
+		)
+		(property "Engineering_Note" "ST BD140, May2008 Rev5 Fig1/p7 drawing0016114E:1BASE,2COLLECTOR,3EMITTER. Installed drawing face toward board+Y; PCB west3E,center2C,east1B. Footprint rotated180deg about collector. Native pad numbering unchanged;1.3mm drills/1.9mm lands for max0.88x0.63mm leads; stand body2mm above board. Not interchangeable with another vendor pinout."
+			(at 0 0 180)
 			(layer "F.SilkS")
 			(hide yes)
@@
 			)
 		)
-		(property "Engineering_Note" "ST1E2C3B,80V1.5A,TO126. ReplacesQCXMPS751mechanismwithoutchangingtopology;betterthermal/SOAdata. HF CWshaper only, NOT VHF AM substitute. MeasurehotSOAandedges."
+		(property "Manufacturer" "STMicroelectronics"
 			(at 0 0 0)
 			(layer "F.SilkS")
@@
 		(duplicate_pad_numbers_are_jumpers no)
 		(fp_line
-			(start -1.83 -2.11)
-			(end 6.39 -2.11)
+			(start 6.39 1.36)
+			(end -1.83 1.36)
 			(stroke
 				(width 0.12)
@@
 		)
 		(fp_line
-			(start -1.83 1.36)
-			(end -1.83 -2.11)
+			(start 6.39 -2.11)
+			(end 6.39 1.36)
 			(stroke
 				(width 0.12)
@@
 		)
 		(fp_line
-			(start 0.68 -2.11)
-			(end 0.68 -1.89)
+			(start 3.88 -2.11)
+			(end 3.88 -1.89)
 			(stroke
 				(width 0.12)
@@
 		)
 		(fp_line
-			(start 3.88 -2.11)
-			(end 3.88 -1.89)
+			(start 0.68 -2.11)
+			(end 0.68 -1.89)
 			(stroke
 				(width 0.12)
@@
 		)
 		(fp_line
-			(start 6.39 -2.11)
-			(end 6.39 1.36)
+			(start -1.83 1.36)
+			(end -1.83 -2.11)
 			(stroke
 				(width 0.12)
@@
 		)
 		(fp_line
-			(start 6.39 1.36)
-			(end -1.83 1.36)
+			(start -1.83 -2.11)
+			(end 6.39 -2.11)
 			(stroke
 				(width 0.12)
@@
 		)
 		(fp_line
-			(start 0.68 -2)
-			(end 0.68 1.25)
+			(start 3.88 -2)
+			(end 3.88 1.25)
 			(stroke
 				(width 0.1)
@@
 		)
 		(fp_line
-			(start 3.88 -2)
-			(end 3.88 1.25)
+			(start 0.68 -2)
+			(end 0.68 1.25)
 			(stroke
 				(width 0.1)
@@
 		)
 		(fp_text user "${REFERENCE}"
-			(at 2.28 -0.38 0)
+			(at 2.28 -0.38 180)
 			(layer "F.Fab")
 			(effects
@@
 		)
 		(pad "1" thru_hole rect
-			(at 0 0)
-			(size 1.71 1.8)
-			(drill 1)
+			(at 0 0 180)
+			(size 1.9 1.9)
+			(drill 1.3)
 			(layers "*.Cu" "*.Mask")
 			(remove_unused_layers no)
-			(net "VPA_LOAD")
+			(net "SHAPE_BASE")
 		)
 		(pad "2" thru_hole oval
-			(at 2.28 0)
-			(size 1.71 1.8)
-			(drill 1)
+			(at 2.28 0 180)
+			(size 1.9 1.9)
+			(drill 1.3)
 			(layers "*.Cu" "*.Mask")
 			(remove_unused_layers no)
@@
 		)
 		(pad "3" thru_hole oval
-			(at 4.56 0)
-			(size 1.71 1.8)
-			(drill 1)
+			(at 4.56 0 180)
+			(size 1.9 1.9)
+			(drill 1.3)
 			(layers "*.Cu" "*.Mask")
 			(remove_unused_layers no)
-			(net "SHAPE_BASE")
+			(net "VPA_LOAD")
 		)
 		(embedded_fonts no)
-		(model "${KICAD10_3DMODEL_DIR}/Package_TO_SOT_THT.3dshapes/TO-126-3_Vertical.step"
+		(model "${KIPRJMOD}/3dmodels/ST_BD140_envelope.wrl"
 			(offset
 				(xyz 0 0 0)
@@
 			)
 		)
-		(property "Engineering_Note" "1 REF,2 anode,3 cathode. >=1mA reference bias; no capacitor directly across TL431 until stability region checked."
+		(property "Engineering_Note" "TI TL431AIDBZR DBZ, SLVS543S May2024 Table5-1/p4:1CATHODE,2REF,3ANODE. E2 corrects E1 anode/reference pad reversal. K andREF tiedVREF_2V5; ANODE ground. Same actual MPN and2.495V functional circuit."
+			(at 0 0 0)
+			(layer "F.SilkS")
+			(hide yes)
+			(effects
+				(font
+					(size 1.27 1.27)
+					(thickness 0.15)
+				)
+			)
+		)
+		(property "Manufacturer" "Texas Instruments"
 			(at 0 0 0)
 			(layer "F.SilkS")
@@
 			(layers "F.Cu" "F.Mask" "F.Paste")
 			(roundrect_rratio 0.25)
-			(net "GND")
+			(net "VREF_2V5")
 		)
 		(pad "3" smd roundrect
@@
 			(layers "F.Cu" "F.Mask" "F.Paste")
 			(roundrect_rratio 0.25)
-			(net "VREF_2V5")
+			(net "GND")
 		)
 		(embedded_fonts no)
@@
 	)
 	(gr_text "Q403"
-		(at 158.28 71.625 0)
+		(at 158.28 72.3 0)
 		(layer "F.SilkS")
 		(effects
@@
 		)
 	)
-	(gr_text "ARDF-TX RF80 / M3B-E1 EVALUATION"
+	(gr_text "ARDF-TX RF80 / M3B-E2 EVALUATION"
 		(at 124 23 0)
 		(layer "F.SilkS")
@@
 		)
 	)
+	(gr_text "3:E     2:C     1:B"
+		(at 158.28 74 0)
+		(layer "F.Fab")
+		(effects
+			(font
+				(size 0.8 0.8)
+				(thickness 0.12)
+			)
+		)
+	)
+	(gr_text "ST BD140: DRAWING FACE TOWARD +Y"
+		(at 158.3 64 0)
+		(layer "F.Fab")
+		(effects
+			(font
+				(size 0.8 0.8)
+				(thickness 0.12)
+			)
+		)
+	)
 	(gr_text "TH301: remote sensor, board pads landing only; see bring-up plan"
 		(at 171 172 0)
@@
 	)
 	(segment
+		(start 107.9375 72)
+		(end 108.8 72)
+		(width 0.28)
+		(layer "F.Cu")
+		(net "GND")
+	)
+	(segment
 		(start 74.525 113.81)
 		(end 74.525 114.81)
@@
 	)
 	(segment
+		(start 108.8 72)
+		(end 108.9 72)
+		(width 0.28)
+		(layer "F.Cu")
+		(net "GND")
+	)
+	(segment
 		(start 160.525 140.81)
 		(end 160.525 141.81)
@@
 	)
 	(segment
-		(start 106.0625 72.95)
-		(end 106.0625 73.95)
-		(width 0.28)
-		(locked yes)
-		(layer "F.Cu")
-		(net "GND")
-	)
-	(segment
 		(start 139.475 35)
 		(end 140.875 35)
@@
 	)
 	(via
+		(at 108.9 72)
+		(size 0.6)
+		(drill 0.3)
+		(layers "F.Cu" "B.Cu")
+		(tenting
+			(front yes)
+			(back yes)
+		)
+		(net "GND")
+	)
+	(via
 		(at 127.675 101)
 		(size 0.6)
@@
 	)
 	(segment
+		(start 107 73)
+		(end 106 73)
+		(width 0.2)
+		(layer "F.Cu")
+		(net "VREF_2V5")
+	)
+	(segment
 		(start 122.175 58)
 		(end 121.6904 58.4846)
@@
 	)
 	(segment
+		(start 106 71)
+		(end 106.0625 71.05)
+		(width 0.2)
+		(layer "F.Cu")
+		(net "VREF_2V5")
+	)
+	(segment
 		(start 106.3257 71.05)
 		(end 107.9484 69.4273)
@@
 	)
 	(segment
-		(start 107.9375 72)
-		(end 107.0125 72)
+		(start 107.9375 73.7056)
+		(end 107.8 73.8)
 		(width 0.2)
 		(layer "F.Cu")
@@
 	)
 	(segment
-		(start 111.175 75)
-		(end 111.175 74.325)
+		(start 106.0625 72.95)
+		(end 106 71)
 		(width 0.2)
 		(layer "F.Cu")
@@
 	)
 	(segment
-		(start 107.0125 72)
-		(end 106.0625 71.05)
+		(start 111.175 75)
+		(end 111.175 74.325)
 		(width 0.2)
 		(layer "F.Cu")
@@
 	)
 	(segment
+		(start 106 73)
+		(end 106.0625 72.95)
+		(width 0.2)
+		(layer "F.Cu")
+		(net "VREF_2V5")
+	)
+	(segment
 		(start 111.175 74.325)
 		(end 111.4287 74.0713)
@@
 	)
 	(segment
+		(start 107.8 73.8)
+		(end 107 73)
+		(width 0.2)
+		(layer "F.Cu")
+		(net "VREF_2V5")
+	)
+	(segment
 		(start 111.4287 74.0713)
 		(end 111.4287 73.3963)
@@
 		(width 0.2)
 		(layer "F.Cu")
-		(net "VREF_2V5")
-	)
-	(segment
-		(start 107.9375 73.7056)
-		(end 107.9375 72)
-		(width 0.2)
-		(layer "F.Cu")
