File: hardware/2m/06_normal_rf.kicad_sch (KiCad schematic)
At the start: 32 parts, among them Q501 PD55008-E, Q502 2N7002, U501 PHA-13HLN+

Commit message: Preserve M5A-R1 VHF electrical candidate and review evidence
Parts:
- added TP604: PA_IN50, TestPoint:TestPoint_Pad_D1.0mm, symbol ARDF_2M:TestPoint
- C605: value 56p -> OPEN 59.6p TUNE; MPN OPEN: C0G100V 56p -> OPEN: OPEN 59.6p TUNE voltage/ESR qualification
- L605: value 27n -> OPEN 28.9n TUNE; MPN 0805HP-27NXJRC -> OPEN: RF tuning inductor OPEN 28.9n TUNE
- Q501: value PD55008-E -> PD54008L-E; symbol ARDF_2M:PD55008_Functional -> ARDF_2M:PD54008_Functional; Engineering_Note Manufacturer Figure1 names G/S/D, not numeric pad order. Fu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 -> PD54008L-E PowerFLAT5x5. Functional G/D/S only until origin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; MPN PD55008-E -> PD54008L-E
- R602: value 53.6 -> 17.8; Engineering_Note 8dB pi pad52.85/116.14 theoretical. Rounded53.6/115; start1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 -> 3dB pi-pad candidate17.6/292.4 theoretical, rounded17.8/287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; MPN RC0603FR-0753R6L -> RC0603FR-0717R8L
- R603, R604: value 115 -> 287; MPN RC0603FR-07115RL -> RC0603FR-07287RL
- RV501: Engineering_Note Pot represented by explicit end/wiper pins. Start wiper grounded. Set Idq <=150mA only after drain rail qualification. -> Pot represented by explicit end/wiper pins. Start wiper grounded. Start Idq50mA; investigate100-200mA only after drain rail qualification.
- U501: value PHA-13HLN+ -> PHA-1+; symbol ARDF_2M:PHA13HLN -> ARDF_2M:PHA1; Engineering_Note DF782:1IN2GND3OUT/DC4paddleGND. Footprint OPEN pending DF78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 -> PHA-1+ DF782:1IN2GND3OUT/DC4paddleGND. Exact landing OPEN.5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; MPN PHA-13HLN+ -> PHA-1+
Connections:
- net PA_IN50: now also TP604.1
- net VDRV_RF: no longer R606.1
- new net VMOD: R606.1
Other:
- note added: "M5A-R1: REVIEW / ALL hardware measurements NOT RUN / no ordering or manufacture."
- note added: "The normal connector has no RF switch or conductor to the training connector. Output matching OPEN: original ST drawing not traced. Do not energize the PA with this assumed-impedance harness. LPF inductors93nH are82nH+11nH in series for current margin and obtainable values."
- note removed: "M5A-R0: REVIEW / ALL hardware measurements NOT RUN / no ordering or manufacture."
- note removed: "The normal connector has no RF switch or conductor to the training connector. Output match is a replaceable 144MHz starting network, not the ST500MHz test network. LPF inductors93nH are82nH+11nH in series for current margin and obtainable values."
