File: hardware/2m/09_test_power.kicad_sch (KiCad schematic)
At the start: 9 parts

Commit message: Preserve M5A-R1 VHF electrical candidate and review evidence
Parts:
- TP904: value VDRV8 -> VDRV_LDO_IN
Connections:
- net VDRV8 renamed VDRV_LDO_IN
Other:
- note added: "M5A-R1: REVIEW / ALL hardware measurements NOT RUN / no ordering or manufacture."
- note added: "No RF2M PCB exists in M5A-R1. All RF/thermal/safety tests NOT_RUN. PWR_FLAG declares a measured external source; it does not validate protection or a supply rating. Read OPEN items in docs/M5A_R1_SCHEMATIC_REVIEW.md before an evaluation PCB."
- note removed: "M5A-R0: REVIEW / ALL hardware measurements NOT RUN / no ordering or manufacture."
- note removed: "No PCB exists in M5A. All RF/thermal/safety tests NOT_RUN. PWR_FLAG declares a measured external source; it does not validate protection or a supply rating. Read OPEN items in docs/M5_2M_SCHEMATIC_REVIEW.md before an evaluation PCB."
