File: hardware/2m/03_input_power.kicad_sch (KiCad schematic)
At the start: 30 parts, among them J301 Protected pack, J302 Exclusive converter link, Q301 2N7002, Q302 AO3401A, Q305 AO3401A, Q306 MMBT3904,215, Q309 AO3401A, U301 TPS54302DDCR, U304 SN74LVC2G08DCUR

Commit message: Preserve M5A-R1 VHF electrical candidate and review evidence
Parts:
- F301: value 2A fast / verify I2t -> 4A fast / qualify I2t; Engineering_Note (none) -> Littelfuse466series32VAC/DC50Ainterrupt,1206,4A code004. Ca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; MPN OPEN 2A fuse with DC interruption rating -> 0466004.NRHF
- R301: value 158k -> 116k; MPN RC0603FR-07158KL -> RC0603FR-07116KL
- R303: value 27k -> 27.8k; MPN RC0603FR-0727KL -> RC0603FR-0727K8L
Other:
- note added: "M5A-R1: REVIEW / ALL hardware measurements NOT RUN / no ordering or manufacture."
- note removed: "M5A-R0: REVIEW / ALL hardware measurements NOT RUN / no ordering or manufacture."

Commit message: Preserve M5A-R3 historical transmitter schematic and review
Parts:
- F301: Engineering_Note Littelfuse466series32VAC/DC50Ainterrupt,1206,4A code004. Ca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 -> Wiring/secondary protection only; 4A fuse does not protect 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
- R301: value 116k -> 171k; Engineering_Note (none) -> Buck reduced10.7876V nominal. Full PROFILE_Q shunts34k into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; MPN RC0603FR-07116KL -> RC0603FR-07171KL
- R303: value 27.8k -> 34k; MPN RC0603FR-0727K8L -> RC0603FR-0734KL
- U304: Engineering_Note Direct comparator logic-low to defined NPN-base low; replac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 -> R3: physical5/6->3 RAIL_RUN requires NORMAL_PERMIT and HARD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
Connections:
- net CONV_EN: no longer U304.5 (2A)
- new net NORMAL_PERMIT: U304.5 (2A)
Other:
- note added: "M5A-R3: REVIEW / ALL hardware measurements NOT RUN / no ordering or manufacture."
- note added: "R3: no RF/analog/thermal hardware validation. Original RF attribution and open procurement in M5A_R3 documents."
- note removed: "J301: 2S 6.0-8.4V for BOOST population OR 4S 12.0-16.8V for BUCK population. Never fit both J302 straps. Pack/window component population is a hardware configuration, not automatic universal routing."
- note removed: "M5A-R1: REVIEW / ALL hardware measurements NOT RUN / no ordering or manufacture."

Commit message: Preserve M5A-R4 economical VHF electrical review baseline
Parts:
- F301: Engineering_Note Wiring/secondary protection only; 4A fuse does not protect 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 -> Littelfuse466series32VAC/DC50Ainterrupt,1206,4A code004. Ca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
- R301: value 171k -> 116k; Engineering_Note Buck reduced10.7876V nominal. Full PROFILE_Q shunts34k into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 -> R4 4S buck7.5096V reduced;capturedPROFILE_Q shunts46.4k ->8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; MPN RC0603FR-07171KL -> RC0603FR-07116KL
- R303: value 34k -> 46.4k; MPN RC0603FR-0734KL -> RC0603FR-0746K4L
- U301: Engineering_Note (none) -> Exact DDCR available in cut tape; no3000reel MOQ assumed. R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
- U304: Engineering_Note R3: physical5/6->3 RAIL_RUN requires NORMAL_PERMIT and HARD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 -> 1/2->7 PACK_RUN=CONV_EN&PACK_OK_N;5/6->3 RAIL_RUN=CONV_EN&H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
Connections:
- net NORMAL_PERMIT is gone; now on net CONV_EN: U304.5 (2A)
Other:
- note added: "M5A-R4: REVIEW / ALL hardware measurements NOT RUN / no ordering or manufacture."
- note added: "M5A-R4: hardware measurements NOT_RUN; source/reference and simplification in R4 documents."
- note removed: "M5A-R3: REVIEW / ALL hardware measurements NOT RUN / no ordering or manufacture."
- note removed: "R3: no RF/analog/thermal hardware validation. Original RF attribution and open procurement in M5A_R3 documents."

Commit message: Preserve M5B-E1 integrated RF2M evaluation baseline
Parts:
- J301: value Protected pack -> Protected pack JST VH; footprint (none) -> Connector_JST:JST_VH_B2P-VH_1x02_P3.96mm_Vertical; Engineering_Note (none) -> JST VH polarized locking2pin,3.96mm pitch.1PACK+2GND. VHR-2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; MPN OPEN keyed 2S/4S power connector -> B2P-VH(LF)(SN)
- J302: Engineering_Note 1-2 BOOST (2S); 2-3 BUCK (4S). Never bridge both; DNP other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 -> One3pin2.54mm row with SNT-100-BK-G shunt;factory variant s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; MPN OPEN keyed exclusive shunt -> TSW-103-07-G-S
- L301: footprint Inductor_SMD:L_Bourns_SRR1260 -> ARDF_2M:Bourns_SRP1265A; Engineering_Note Manufacturer family verified.USD0.92 family price /ECB1.119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 -> Bourns SRP1265A10uH shielded family;manufacturer12.5mm squa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; MPN OPEN: shielded power inductor 10u -> SRP1265A-100M
Other:
- note added: "M5B-E1 / integrated evaluation PCB / NOT RELEASED / hardware tests NOT_RUN"
- note added: "M5B-E1: REVIEW / ALL hardware measurements NOT RUN / no ordering or manufacture."
- note removed: "M5A-R4: REVIEW / ALL hardware measurements NOT RUN / no ordering or manufacture."
- note removed: "M5A-R4: hardware measurements NOT_RUN; source/reference and simplification in R4 documents."

Commit message: Implement M5B-E3 standard JLCPCB RF2M evaluation board
Recalculate and implement 1.6 mm / 1 oz RF geometry, power copper, thermal vias, connector holes and manufacturing legend. Preserve electrical functions and population variants. Add native-geometry DFM, regression checks and fresh native/fabrication review archives. CAD milestone only; no manufacturing or operational release.
Parts:
- C301, C304, C305: footprint Capacitor_SMD:C_1210_3225Metric -> ARDF_2M:C_1210_3225Metric_E3
- C302, C303, C310: footprint Capacitor_SMD:C_0603_1608Metric -> ARDF_2M:C_0603_1608Metric_E3
- D302: footprint Diode_SMD:D_SMB -> ARDF_2M:D_SMB_E3
- D306, D307: footprint Diode_SMD:D_SOD-123F -> ARDF_2M:D_SOD-123F_E3
- F301: footprint Fuse:Fuse_1206_3216Metric -> ARDF_2M:Fuse_1206_3216Metric_E3
- J301: footprint Connector_JST:JST_VH_B2P-VH_1x02_P3.96mm_Vertical -> ARDF_2M:JST_VH_B2P-VH_1x02_P3.96mm_Vertical_E3; Engineering_Note JST VH polarized locking2pin,3.96mm pitch.1PACK+2GND. VHR-2N housing/SVH contacts;strain-relief harness to board support. Different charger interface required. Hardware pack window precedes converter feed;never assume connector identifies cell count. -> JST VH polarized locking2pin,3.96mm pitch.1PACK+2GND. VHR-2N housing/SVH contacts;strain-relief harness to board support. Different charger interface required. Hardware pack window precedes converter feed;never assume connector identifies cell count. E3:1.80mmfinishedhole(retainland),JLCminimum1.72mmversusnominal1.14mmsquarelead1.612mmdiagonal. JSTspecifies1.6mmboard;incomingfit/polarityinspectionrequired.
- J302: footprint Connector_PinHeader_2.54mm:PinHeader_1x03_P2.54mm_Vertical -> ARDF_2M:PinHeader_1x03_P2.54mm_Vertical_E3
- Q301, Q302, Q305, Q306, Q309: footprint Package_TO_SOT_SMD:SOT-23 -> ARDF_2M:SOT-23_E3
- R301, R302, R303, R304, R305, R310, R311, R312, R313, R314: footprint Resistor_SMD:R_0603_1608Metric -> ARDF_2M:R_0603_1608Metric_E3
- U301: footprint Package_TO_SOT_SMD:SOT-23-6_Handsoldering -> ARDF_2M:SOT-23-6_Handsoldering_E3
- U304: footprint Package_SO:VSSOP-8_2.3x2mm_P0.5mm -> ARDF_2M:VSSOP-8_2.3x2mm_P0.5mm_E3
Other:
- note added: "M5B-E3 / integrated evaluation PCB / NOT RELEASED / hardware tests NOT_RUN"
- note added: "M5B-E3: REVIEW / ALL hardware measurements NOT RUN / no ordering or manufacture."
- note removed: "M5B-E1 / integrated evaluation PCB / NOT RELEASED / hardware tests NOT_RUN"
- note removed: "M5B-E1: REVIEW / ALL hardware measurements NOT RUN / no ordering or manufacture."

Commit message: Implement M5B-E4 thermal candidate with source-joint assembly hold
Other:
- note added: "M5B-E4 / integrated evaluation PCB / NOT RELEASED / hardware tests NOT_RUN"
- note added: "M5B-E4: REVIEW / ALL hardware measurements NOT RUN / no ordering or manufacture."
- note removed: "M5B-E3 / integrated evaluation PCB / NOT RELEASED / hardware tests NOT_RUN"
- note removed: "M5B-E3: REVIEW / ALL hardware measurements NOT RUN / no ordering or manufacture."

Commit message: Implement M5B-E4R1 source-joint prototype candidate
Replace source mask islands with a controlled open-via hybrid and native-derived local stencil. Preserve standard JLCPCB and RF circuitry. Add assembly qualification, thermal convergence and adverse sensitivities, native DFM/mutation checks and fresh review exports. Conservative 110 C target is missed; 125 C physical gate stays open. No acceptance tag or manufacturing authorization.
Other:
- note added: "M5B-E4R1R1R1 / integrated evaluation PCB / NOT RELEASED / hardware tests NOT_RUN"
- note added: "M5B-E4R1R1R1: REVIEW / ALL hardware measurements NOT RUN / no ordering or manufacture."
- note removed: "M5B-E4 / integrated evaluation PCB / NOT RELEASED / hardware tests NOT_RUN"
- note removed: "M5B-E4: REVIEW / ALL hardware measurements NOT RUN / no ordering or manufacture."

Commit message: M5B-E5: compact RF2M to the shared 150x110 mm platform
Other:
- note added: "M5B-E5R1R1 / integrated evaluation PCB / NOT RELEASED / hardware tests NOT_RUN"
- note added: "M5B-E5R1R1: REVIEW / ALL hardware measurements NOT RUN / no ordering or manufacture."
- note removed: "M5B-E4R1R1R1 / integrated evaluation PCB / NOT RELEASED / hardware tests NOT_RUN"
- note removed: "M5B-E4R1R1R1: REVIEW / ALL hardware measurements NOT RUN / no ordering or manufacture."
