File: hardware/2m/08_protection.kicad_sch (KiCad schematic)
At the start: 30 parts, among them U801 TL431BIDBZR, U804 INA180A1IDBVR

Commit message: Preserve M5A-R1 VHF electrical candidate and review evidence
Parts:
- R807: Engineering_Note 2S58.3k gives6.210V raw UV. BUCK4S24.9k gives12.15V reduced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 -> 2S58.3k gives6.210V raw UV. BUCK4S24.9k gives12.15V for bot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
- R813: value 12.4k -> 20.9k; MPN RC0603FR-0712K4L -> RC0603FR-0720K9L
- R817: value 15.4k -> 29.4k; MPN RC0603FR-0715K4L -> RC0603FR-0729K4L
- R821: value 13.7k -> 26.5k; Engineering_Note VPA overvoltage12.63V nominal: catches pass E-C short indep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 -> VPA overvoltage8.20V nominal: catches pass E-C short indepe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; MPN RC0603FR-0713K7L -> RC0603FR-0726K5L
- U804: Engineering_Note A1gain20 x0.1ohm =>2V/A; ISENSE divider10k/7.5k against loa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 -> A1gain20 x0.1ohm =>2V/A; ISENSE divider10k/4.02k against lo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
Other:
- note added: "M5A-R1: REVIEW / ALL hardware measurements NOT RUN / no ordering or manufacture."
- note removed: "M5A-R0: REVIEW / ALL hardware measurements NOT RUN / no ordering or manufacture."

Commit message: Preserve M5A-R3 historical transmitter schematic and review
Parts:
- removed R815: 80.6k, Resistor_SMD:R_0603_1608Metric, symbol ARDF_2M:R
- removed R816, R818: 10k, Resistor_SMD:R_0603_1608Metric, symbol ARDF_2M:R
- removed R817: 29.4k, Resistor_SMD:R_0603_1608Metric, symbol ARDF_2M:R
- R811: value 120k -> 160k; MPN RC0603FR-07120KL -> RC0603FR-07160KL
- R813: value 20.9k -> 18.2k; MPN RC0603FR-0720K9L -> RC0603FR-0718K2L
- R819: value 110k -> 160k; MPN RC0603FR-07110KL -> RC0603FR-07160KL
- R821: value 26.5k -> 18.2k; MPN RC0603FR-0726K5L -> RC0603FR-0718K2L
Other:
- note added: "M5A-R3: REVIEW / ALL hardware measurements NOT RUN / no ordering or manufacture."
- note added: "R3: no RF/analog/thermal hardware validation. Original RF attribution and open procurement in M5A_R3 documents."
- note removed: "Analog faults only affect normal PA population; training uses bounded3.3V and protected host pack. Eight comparators, one current amplifier, one common reference: distinct voltage/current/sensor functions. No permanent RF detector or ADC."
- note removed: "M5A-R1: REVIEW / ALL hardware measurements NOT RUN / no ordering or manufacture."

Commit message: Preserve M5A-R4 economical VHF electrical review baseline
Parts:
- added R815: 75k, Resistor_SMD:R_0603_1608Metric, symbol ARDF_2M:R
- added R816, R818: 10k, Resistor_SMD:R_0603_1608Metric, symbol ARDF_2M:R
- added R817: 29.4k, Resistor_SMD:R_0603_1608Metric, symbol ARDF_2M:R
- R811: value 160k -> 120k; Engineering_Note (none) -> Raw upstream rail sense; controller confirms settled9V befo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; MPN RC0603FR-07160KL -> RC0603FR-07120KL
- R813: value 18.2k -> 20.9k; MPN RC0603FR-0718K2L -> RC0603FR-0720K9L
- R819: value 160k -> 110k; MPN RC0603FR-07160KL -> RC0603FR-07110KL
- R821: value 18.2k -> 26.5k; MPN RC0603FR-0718K2L -> RC0603FR-0726K5L
Connections:
- net GND: now also R816.2, R818.2
- net VREF2V5: now also R817.1
- new net DRV_OV_REF: R817.2, R818.1
- new net DRV_S: R815.2, R816.1
- new net VDRV_FILTER: R815.1
Other:
- note added: "M5A-R4: REVIEW / ALL hardware measurements NOT RUN / no ordering or manufacture."
- note added: "M5A-R4: hardware measurements NOT_RUN; source/reference and simplification in R4 documents."
- note removed: "M5A-R3: REVIEW / ALL hardware measurements NOT RUN / no ordering or manufacture."
- note removed: "R3: no RF/analog/thermal hardware validation. Original RF attribution and open procurement in M5A_R3 documents."

Commit message: Preserve M5B-E1 integrated RF2M evaluation baseline
Parts:
- R815: value 75k -> 73.2k; Engineering_Note R4 driver OV divider:0.1percent thin film required, not1per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 -> 0.1percent driver OV divider;nominal5.269V with originalref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; MPN RT0603BRD0775KL -> RT0603BRD0773K2L
- TH801: value 10k NTC B3950 -> 10k NTC B3977; footprint Resistor_THT:R_Axial_DIN0207_L6.3mm_D2.5mm_P7.62mm_Horizontal -> ARDF_2M:NTC_Remote_2Wire; Engineering_Note Bond to PA/modulator thermal spreader; open and short detec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 -> Vishay10k25C bead B25/853977K,not3950. Insulated wires to p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; MPN OPEN insulated contact NTC10k B3950 -> NTCLE100E3103JB0
Other:
- note added: "M5B-E1 / integrated evaluation PCB / NOT RELEASED / hardware tests NOT_RUN"
- note added: "M5B-E1: REVIEW / ALL hardware measurements NOT RUN / no ordering or manufacture."
- note removed: "M5A-R4: REVIEW / ALL hardware measurements NOT RUN / no ordering or manufacture."
- note removed: "M5A-R4: hardware measurements NOT_RUN; source/reference and simplification in R4 documents."

Commit message: Implement M5B-E3 standard JLCPCB RF2M evaluation board
Recalculate and implement 1.6 mm / 1 oz RF geometry, power copper, thermal vias, connector holes and manufacturing legend. Preserve electrical functions and population variants. Add native-geometry DFM, regression checks and fresh native/fabrication review archives. CAD milestone only; no manufacturing or operational release.
Parts:
- R801, R802, R803, R804, R805, R806, R807, R808, R809, R810, R811, R812, R813, R814, R815, R816, R817, R818, R819, R820, R821, R822, R823, R824, R825, R826, R827: footprint Resistor_SMD:R_0603_1608Metric -> ARDF_2M:R_0603_1608Metric_E3
- U801: footprint Package_TO_SOT_SMD:SOT-23 -> ARDF_2M:SOT-23_E3
- U804: footprint Package_TO_SOT_SMD:SOT-23-5 -> ARDF_2M:SOT-23-5_E3
Other:
- note added: "M5B-E3 / integrated evaluation PCB / NOT RELEASED / hardware tests NOT_RUN"
- note added: "M5B-E3: REVIEW / ALL hardware measurements NOT RUN / no ordering or manufacture."
- note removed: "M5B-E1 / integrated evaluation PCB / NOT RELEASED / hardware tests NOT_RUN"
- note removed: "M5B-E1: REVIEW / ALL hardware measurements NOT RUN / no ordering or manufacture."

Commit message: Implement M5B-E4 thermal candidate with source-joint assembly hold
Other:
- note added: "M5B-E4 / integrated evaluation PCB / NOT RELEASED / hardware tests NOT_RUN"
- note added: "M5B-E4: REVIEW / ALL hardware measurements NOT RUN / no ordering or manufacture."
- note removed: "M5B-E3 / integrated evaluation PCB / NOT RELEASED / hardware tests NOT_RUN"
- note removed: "M5B-E3: REVIEW / ALL hardware measurements NOT RUN / no ordering or manufacture."

Commit message: Implement M5B-E4R1 source-joint prototype candidate
Replace source mask islands with a controlled open-via hybrid and native-derived local stencil. Preserve standard JLCPCB and RF circuitry. Add assembly qualification, thermal convergence and adverse sensitivities, native DFM/mutation checks and fresh review exports. Conservative 110 C target is missed; 125 C physical gate stays open. No acceptance tag or manufacturing authorization.
Other:
- note added: "M5B-E4R1R1R1 / integrated evaluation PCB / NOT RELEASED / hardware tests NOT_RUN"
- note added: "M5B-E4R1R1R1: REVIEW / ALL hardware measurements NOT RUN / no ordering or manufacture."
- note removed: "M5B-E4 / integrated evaluation PCB / NOT RELEASED / hardware tests NOT_RUN"
- note removed: "M5B-E4: REVIEW / ALL hardware measurements NOT RUN / no ordering or manufacture."

Commit message: M5B-E5: compact RF2M to the shared 150x110 mm platform
Other:
- note added: "M5B-E5R1R1 / integrated evaluation PCB / NOT RELEASED / hardware tests NOT_RUN"
- note added: "M5B-E5R1R1: REVIEW / ALL hardware measurements NOT RUN / no ordering or manufacture."
- note removed: "M5B-E4R1R1R1 / integrated evaluation PCB / NOT RELEASED / hardware tests NOT_RUN"
- note removed: "M5B-E4R1R1R1: REVIEW / ALL hardware measurements NOT RUN / no ordering or manufacture."
