File: hardware/2m/08_protectionb1.kicad_sch (KiCad schematic)
At the start: 19 parts, among them Q801 2N7002, U802 LM339BDR, U803 LM339BDR

Commit message: Preserve M5A-R1 VHF electrical candidate and review evidence
Parts:
- removed Q801: 2N7002, Package_TO_SOT_SMD:SOT-23, symbol ARDF_2M:2N7002
- removed R830: 84.5k, Resistor_SMD:R_0603_1608Metric, symbol ARDF_2M:R
- R829: value 7.5k -> 4.02k; MPN RC0603FR-077K5L -> RC0603FR-074K02L
Other:
- note added: "M5A-R1: REVIEW / ALL hardware measurements NOT RUN / no ordering or manufacture."
- note removed: "M5A-R0: REVIEW / ALL hardware measurements NOT RUN / no ordering or manufacture."
- moved on the sheet: C104, C801, C802, C803, C804, D801, D802, R117, R118, R828, R829, R832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

Commit message: Preserve M5A-R3 historical transmitter schematic and review
Parts:
- R828: value 10k -> 1.5k; Engineering_Note (none) -> R3 total normal-rail current trip approximately0.593A using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; MPN RC0603FR-0710KL -> RC0603FR-071K5L
- R829: value 4.02k -> 10k; MPN RC0603FR-074K02L -> RC0603FR-0710KL
- U802: Engineering_Note 3.3V; reference nodes below1.135V hot common-mode limit at3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 -> R3 unused former MMIC-OV comparator tied to valid common-mo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
- U803: Engineering_Note 3.3V; reference nodes below1.135V hot common-mode limit at3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 -> R3: approximately0.593A current trip; original ~66C NTC win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
Connections:
- net DRV_OV_REF is gone; now on net VREF1V0: U802.9 (+)
- net DRV_S is gone; now on net GND: U802.8 (-)
Other:
- note added: "M5A-R3: REVIEW / ALL hardware measurements NOT RUN / no ordering or manufacture."
- note added: "R3: no RF/analog/thermal hardware validation. Original RF attribution and open procurement in M5A_R3 documents."
- note removed: "M5A-R1: REVIEW / ALL hardware measurements NOT RUN / no ordering or manufacture."

Commit message: Preserve M5A-R4 economical VHF electrical review baseline
Parts:
- R828: value 1.5k -> 10k; Engineering_Note R3 total normal-rail current trip approximately0.593A using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 -> (none); MPN RC0603FR-071K5L -> RC0603FR-0710KL
- R829: value 10k -> 4.02k; MPN RC0603FR-0710KL -> RC0603FR-074K02L
- U802: Engineering_Note R3 unused former MMIC-OV comparator tied to valid common-mo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 -> 3.3V; reference nodes below1.135V hot common-mode limit at3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
- U803: Engineering_Note R3: approximately0.593A current trip; original ~66C NTC win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 -> 3.3V; reference nodes below1.135V hot common-mode limit at3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
Connections:
- net GND: no longer U802.8 (-)
- net VREF1V0: no longer U802.9 (+)
- new net DRV_OV_REF: U802.9 (+)
- new net DRV_S: U802.8 (-)
Other:
- note added: "M5A-R4: REVIEW / ALL hardware measurements NOT RUN / no ordering or manufacture."
- note added: "M5A-R4: hardware measurements NOT_RUN; source/reference and simplification in R4 documents."
- note removed: "M5A-R3: REVIEW / ALL hardware measurements NOT RUN / no ordering or manufacture."
- note removed: "R3: no RF/analog/thermal hardware validation. Original RF attribution and open procurement in M5A_R3 documents."

Commit message: Preserve M5B-E1 integrated RF2M evaluation baseline
Parts:
- R828: value 10k -> 5.11k; Engineering_Note (none) -> 0.1percent current-sense divider upper resistor. With4.02k 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; MPN RC0603FR-0710KL -> RT0603BRD075K11L
Other:
- note added: "M5B-E1 / integrated evaluation PCB / NOT RELEASED / hardware tests NOT_RUN"
- note added: "M5B-E1: REVIEW / ALL hardware measurements NOT RUN / no ordering or manufacture."
- note removed: "M5A-R4: REVIEW / ALL hardware measurements NOT RUN / no ordering or manufacture."
- note removed: "M5A-R4: hardware measurements NOT_RUN; source/reference and simplification in R4 documents."

Commit message: Implement M5B-E3 standard JLCPCB RF2M evaluation board
Recalculate and implement 1.6 mm / 1 oz RF geometry, power copper, thermal vias, connector holes and manufacturing legend. Preserve electrical functions and population variants. Add native-geometry DFM, regression checks and fresh native/fabrication review archives. CAD milestone only; no manufacturing or operational release.
Parts:
- C104, C801, C802, C803, C804: footprint Capacitor_SMD:C_0603_1608Metric -> ARDF_2M:C_0603_1608Metric_E3
- D801, D802: footprint Diode_SMD:D_SOD-323 -> ARDF_2M:D_SOD-323_E3
- R117, R118, R828, R829, R832, R833: footprint Resistor_SMD:R_0603_1608Metric -> ARDF_2M:R_0603_1608Metric_E3
- TP801, TP802: footprint TestPoint:TestPoint_Pad_D1.0mm -> ARDF_2M:TestPoint_Pad_D1.0mm_E3
- U802, U803: footprint Package_SO:SOIC-14_3.9x8.7mm_P1.27mm -> ARDF_2M:SOIC-14_3.9x8.7mm_P1.27mm_E3
Other:
- note added: "M5B-E3 / integrated evaluation PCB / NOT RELEASED / hardware tests NOT_RUN"
- note added: "M5B-E3: REVIEW / ALL hardware measurements NOT RUN / no ordering or manufacture."
- note removed: "M5B-E1 / integrated evaluation PCB / NOT RELEASED / hardware tests NOT_RUN"
- note removed: "M5B-E1: REVIEW / ALL hardware measurements NOT RUN / no ordering or manufacture."

Commit message: Implement M5B-E4 thermal candidate with source-joint assembly hold
Other:
- note added: "M5B-E4 / integrated evaluation PCB / NOT RELEASED / hardware tests NOT_RUN"
- note added: "M5B-E4: REVIEW / ALL hardware measurements NOT RUN / no ordering or manufacture."
- note removed: "M5B-E3 / integrated evaluation PCB / NOT RELEASED / hardware tests NOT_RUN"
- note removed: "M5B-E3: REVIEW / ALL hardware measurements NOT RUN / no ordering or manufacture."

Commit message: Implement M5B-E4R1 source-joint prototype candidate
Replace source mask islands with a controlled open-via hybrid and native-derived local stencil. Preserve standard JLCPCB and RF circuitry. Add assembly qualification, thermal convergence and adverse sensitivities, native DFM/mutation checks and fresh review exports. Conservative 110 C target is missed; 125 C physical gate stays open. No acceptance tag or manufacturing authorization.
Other:
- note added: "M5B-E4R1R1R1 / integrated evaluation PCB / NOT RELEASED / hardware tests NOT_RUN"
- note added: "M5B-E4R1R1R1: REVIEW / ALL hardware measurements NOT RUN / no ordering or manufacture."
- note removed: "M5B-E4 / integrated evaluation PCB / NOT RELEASED / hardware tests NOT_RUN"
- note removed: "M5B-E4: REVIEW / ALL hardware measurements NOT RUN / no ordering or manufacture."

Commit message: M5B-E5: compact RF2M to the shared 150x110 mm platform
Other:
- note added: "M5B-E5R1R1 / integrated evaluation PCB / NOT RELEASED / hardware tests NOT_RUN"
- note added: "M5B-E5R1R1: REVIEW / ALL hardware measurements NOT RUN / no ordering or manufacture."
- note removed: "M5B-E4R1R1R1 / integrated evaluation PCB / NOT RELEASED / hardware tests NOT_RUN"
- note removed: "M5B-E4R1R1R1: REVIEW / ALL hardware measurements NOT RUN / no ordering or manufacture."
