File: hardware/2m/04_boost_driver_supply.kicad_sch (KiCad schematic)
At the start: 19 parts, among them U302 TPS611781RNWR, U303 TLV76150DCYR

Commit message: Preserve M5B-E1 integrated RF2M evaluation baseline
Parts:
- C406: Engineering_Note Starting compensation, not validated for selected L/C/load. -> Starting compensation, not validated for selected L/C/load.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; MPN OPEN: 0603 C0G50V 100p -> CC0603JRNPO9BN101
- C409: footprint (none) -> ARDF_2M:CP_Panasonic_OSCON_C10; Engineering_Note Panasonic25SVPG150M150uF25V+/-20percent,ESR13mohm@100kHz,4.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 -> Panasonic C10 land a2.1 b9.1 c1.6mm;150u25V+/-20,13mohm100k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
- L302: footprint Inductor_SMD:L_Bourns_SRR1260 -> ARDF_2M:Bourns_SRP1265A; Engineering_Note Manufacturer family verified.USD0.92 family price /ECB1.119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 -> Bourns SRP1265A4.7uH shielded,manufacturer landing;2S boost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; MPN OPEN: shielded power inductor 4.7u -> SRP1265A-4R7M
- R413: value 8.2 -> 4.7; Engineering_Note 0.266W at180mA;initial reservoir current<=1.14A at9.2V/8.11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 -> 4.7ohm1W feed before two independent regulators. Precharge/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; MPN OPEN:8.2ohm1percent1W2512 -> RC2512FK-074R7L
- U303: Engineering_Note Fixed5V TI DCY1GND2OUT/tab3IN. After8.2ohm at180mA input~7.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 -> Existing TLV76150 fixed5V is second independent regulation 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
Connections:
- net VDRV_LDO_IN: no longer U303.3 (IN)
- new net VDRV_PREREG: U303.3 (IN)
Other:
- note added: "M5B-E1 / integrated evaluation PCB / NOT RELEASED / hardware tests NOT_RUN"
- note added: "M5B-E1: REVIEW / ALL hardware measurements NOT RUN / no ordering or manufacture."
- note removed: "M5A-R4: REVIEW / ALL hardware measurements NOT RUN / no ordering or manufacture."
- note removed: "M5A-R4: hardware measurements NOT_RUN; source/reference and simplification in R4 documents."

Commit message: Implement M5B-E3 standard JLCPCB RF2M evaluation board
Recalculate and implement 1.6 mm / 1 oz RF geometry, power copper, thermal vias, connector holes and manufacturing legend. Preserve electrical functions and population variants. Add native-geometry DFM, regression checks and fresh native/fabrication review archives. CAD milestone only; no manufacturing or operational release.
Parts:
- C401, C405, C406: footprint Capacitor_SMD:C_0603_1608Metric -> ARDF_2M:C_0603_1608Metric_E3
- C402: footprint Capacitor_SMD:C_1206_3216Metric -> ARDF_2M:C_1206_3216Metric_E3
- C403, C404: footprint Capacitor_SMD:C_1210_3225Metric -> ARDF_2M:C_1210_3225Metric_E3
- C407: footprint Capacitor_SMD:C_0805_2012Metric -> ARDF_2M:C_0805_2012Metric_E3
- D309: footprint Diode_SMD:D_SMA -> ARDF_2M:D_SMA_E3
- R401, R402, R403, R404, R405: footprint Resistor_SMD:R_0603_1608Metric -> ARDF_2M:R_0603_1608Metric_E3
- R413: footprint Resistor_SMD:R_2512_6332Metric -> ARDF_2M:R_2512_6332Metric_E3
- TP401: footprint TestPoint:TestPoint_Pad_D1.0mm -> ARDF_2M:TestPoint_Pad_D1.0mm_E3
- U303: footprint Package_TO_SOT_SMD:SOT-223-3_TabPin2 -> ARDF_2M:SOT-223-3_TabPin2_E3
Other:
- note added: "M5B-E3 / integrated evaluation PCB / NOT RELEASED / hardware tests NOT_RUN"
- note added: "M5B-E3: REVIEW / ALL hardware measurements NOT RUN / no ordering or manufacture."
- note removed: "M5B-E1 / integrated evaluation PCB / NOT RELEASED / hardware tests NOT_RUN"
- note removed: "M5B-E1: REVIEW / ALL hardware measurements NOT RUN / no ordering or manufacture."

Commit message: Implement M5B-E4 thermal candidate with source-joint assembly hold
Other:
- note added: "M5B-E4 / integrated evaluation PCB / NOT RELEASED / hardware tests NOT_RUN"
- note added: "M5B-E4: REVIEW / ALL hardware measurements NOT RUN / no ordering or manufacture."
- note removed: "M5B-E3 / integrated evaluation PCB / NOT RELEASED / hardware tests NOT_RUN"
- note removed: "M5B-E3: REVIEW / ALL hardware measurements NOT RUN / no ordering or manufacture."

Commit message: Implement M5B-E4R1 source-joint prototype candidate
Replace source mask islands with a controlled open-via hybrid and native-derived local stencil. Preserve standard JLCPCB and RF circuitry. Add assembly qualification, thermal convergence and adverse sensitivities, native DFM/mutation checks and fresh review exports. Conservative 110 C target is missed; 125 C physical gate stays open. No acceptance tag or manufacturing authorization.
Other:
- note added: "M5B-E4R1R1R1 / integrated evaluation PCB / NOT RELEASED / hardware tests NOT_RUN"
- note added: "M5B-E4R1R1R1: REVIEW / ALL hardware measurements NOT RUN / no ordering or manufacture."
- note removed: "M5B-E4 / integrated evaluation PCB / NOT RELEASED / hardware tests NOT_RUN"
- note removed: "M5B-E4: REVIEW / ALL hardware measurements NOT RUN / no ordering or manufacture."

Commit message: M5B-E5: compact RF2M to the shared 150x110 mm platform
Other:
- note added: "M5B-E5R1R1 / integrated evaluation PCB / NOT RELEASED / hardware tests NOT_RUN"
- note added: "M5B-E5R1R1: REVIEW / ALL hardware measurements NOT RUN / no ordering or manufacture."
- note removed: "M5B-E4R1R1R1 / integrated evaluation PCB / NOT RELEASED / hardware tests NOT_RUN"
- note removed: "M5B-E4R1R1R1: REVIEW / ALL hardware measurements NOT RUN / no ordering or manufacture."

Commit message: M5B-E6R2: Implement carrier-keyed RF2M and unified cooling
Other:
- note added: "M5B-E6R2 / integrated evaluation PCB / NOT RELEASED / hardware tests NOT_RUN"
- note added: "M5B-E6R2: REVIEW / ALL hardware measurements NOT RUN / no ordering or manufacture."
- note removed: "M5B-E5R1R1 / integrated evaluation PCB / NOT RELEASED / hardware tests NOT_RUN"
- note removed: "M5B-E5R1R1: REVIEW / ALL hardware measurements NOT RUN / no ordering or manufacture."
