File: hardware/2m/05_am.kicad_sch (KiCad schematic)
At the start: 30 parts, among them Q401 D45H11, Q402 BD139, Q403 MMBT3904,215, Q404 MMBT3904,215, Q405 MMBT3904,215, U401 TLV9004IDR, U402 SN74LVC1G3157DBVR

Commit message: Preserve M5B-E1 integrated RF2M evaluation baseline
Parts:
- R506: footprint Resistor_SMD:R_2010_5025Metric -> Resistor_SMD:R_2512_6332Metric; Engineering_Note At73mA helper limit:0.053W.1W pulse allowance retained;10oh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 -> 10ohm1W base-path resistor,selected2512 package;not an unqu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; MPN OPEN10ohm1W2010 -> RC2512FK-0710RL
Other:
- note added: "M5B-E1 / integrated evaluation PCB / NOT RELEASED / hardware tests NOT_RUN"
- note added: "M5B-E1: REVIEW / ALL hardware measurements NOT RUN / no ordering or manufacture."
- note removed: "M5A-R4: REVIEW / ALL hardware measurements NOT RUN / no ordering or manufacture."
- note removed: "M5A-R4: hardware measurements NOT_RUN; source/reference and simplification in R4 documents."

Commit message: Implement M5B-E3 standard JLCPCB RF2M evaluation board
Recalculate and implement 1.6 mm / 1 oz RF geometry, power copper, thermal vias, connector holes and manufacturing legend. Preserve electrical functions and population variants. Add native-geometry DFM, regression checks and fresh native/fabrication review archives. CAD milestone only; no manufacturing or operational release.
Parts:
- C501, C502, C503, C504, C505, C506: footprint Capacitor_SMD:C_0603_1608Metric -> ARDF_2M:C_0603_1608Metric_E3
- Q401: footprint Package_TO_SOT_THT:TO-220-3_Vertical -> ARDF_2M:TO-220-3_Vertical_E3
- Q402: footprint Package_TO_SOT_THT:TO-126-3_Vertical -> ARDF_2M:TO-126-3_Vertical_E3
- Q403, Q404, Q405: footprint Package_TO_SOT_SMD:SOT-23 -> ARDF_2M:SOT-23_E3
- R501, R502, R503, R504, R505, R508, R509, R510, R511, R512, R514, R516, R517, R518: footprint Resistor_SMD:R_0603_1608Metric -> ARDF_2M:R_0603_1608Metric_E3
- R506: footprint Resistor_SMD:R_2512_6332Metric -> ARDF_2M:R_2512_6332Metric_E3
- R507: footprint Resistor_SMD:R_0805_2012Metric -> ARDF_2M:R_0805_2012Metric_E3
- R513: footprint Resistor_SMD:R_1206_3216Metric -> ARDF_2M:R_1206_3216Metric_E3
- U401: footprint Package_SO:SOIC-14_3.9x8.7mm_P1.27mm -> ARDF_2M:SOIC-14_3.9x8.7mm_P1.27mm_E3
- U402: footprint Package_TO_SOT_SMD:SOT-23-6 -> ARDF_2M:SOT-23-6_E3
Other:
- note added: "M5B-E3 / integrated evaluation PCB / NOT RELEASED / hardware tests NOT_RUN"
- note added: "M5B-E3: REVIEW / ALL hardware measurements NOT RUN / no ordering or manufacture."
- note removed: "M5B-E1 / integrated evaluation PCB / NOT RELEASED / hardware tests NOT_RUN"
- note removed: "M5B-E1: REVIEW / ALL hardware measurements NOT RUN / no ordering or manufacture."

Commit message: Implement M5B-E4 thermal candidate with source-joint assembly hold
Other:
- note added: "M5B-E4 / integrated evaluation PCB / NOT RELEASED / hardware tests NOT_RUN"
- note added: "M5B-E4: REVIEW / ALL hardware measurements NOT RUN / no ordering or manufacture."
- note removed: "M5B-E3 / integrated evaluation PCB / NOT RELEASED / hardware tests NOT_RUN"
- note removed: "M5B-E3: REVIEW / ALL hardware measurements NOT RUN / no ordering or manufacture."

Commit message: Implement M5B-E4R1 source-joint prototype candidate
Replace source mask islands with a controlled open-via hybrid and native-derived local stencil. Preserve standard JLCPCB and RF circuitry. Add assembly qualification, thermal convergence and adverse sensitivities, native DFM/mutation checks and fresh review exports. Conservative 110 C target is missed; 125 C physical gate stays open. No acceptance tag or manufacturing authorization.
Other:
- note added: "M5B-E4R1R1R1 / integrated evaluation PCB / NOT RELEASED / hardware tests NOT_RUN"
- note added: "M5B-E4R1R1R1: REVIEW / ALL hardware measurements NOT RUN / no ordering or manufacture."
- note removed: "M5B-E4 / integrated evaluation PCB / NOT RELEASED / hardware tests NOT_RUN"
- note removed: "M5B-E4: REVIEW / ALL hardware measurements NOT RUN / no ordering or manufacture."

Commit message: M5B-E5: compact RF2M to the shared 150x110 mm platform
Other:
- note added: "M5B-E5R1R1 / integrated evaluation PCB / NOT RELEASED / hardware tests NOT_RUN"
- note added: "M5B-E5R1R1: REVIEW / ALL hardware measurements NOT RUN / no ordering or manufacture."
- note removed: "M5B-E4R1R1R1 / integrated evaluation PCB / NOT RELEASED / hardware tests NOT_RUN"
- note removed: "M5B-E4R1R1R1: REVIEW / ALL hardware measurements NOT RUN / no ordering or manufacture."

Commit message: M5B-E6R2: Implement carrier-keyed RF2M and unified cooling
Parts:
- Q401: footprint ARDF_2M:TO-220-3_Vertical_E3 -> ARDF_2M:TO220_Flat_CommonPlane_E6R2
- Q402: footprint ARDF_2M:TO-126-3_Vertical_E3 -> ARDF_2M:TO126_Flat_CommonPlane_E6R2
Connections:
- net GND: now also U402.3 (B1_KEY0)
- net LEVEL_DC: no longer U402.3 (B1_KEY0)
- net MOD_OFF_BASE: no longer Q405.1 (B)
- net VPA: no longer Q401.2 (C)
- net NORMAL_OFF renamed LOCAL_MOD_OFF
- new net MOD_COMMAND_OFF_BASE: Q405.1 (B)
- new net VPA_PRE: Q401.2 (C)
Other:
- note added: "M5B-E6R2 / integrated evaluation PCB / NOT RELEASED / hardware tests NOT_RUN"
- note added: "M5B-E6R2: REVIEW / ALL hardware measurements NOT RUN / no ordering or manufacture."
- note removed: "M5B-E5R1R1 / integrated evaluation PCB / NOT RELEASED / hardware tests NOT_RUN"
- note removed: "M5B-E5R1R1: REVIEW / ALL hardware measurements NOT RUN / no ordering or manufacture."
