File: hardware/2m/05_amb1.kicad_sch (KiCad schematic)
At the start: 6 parts

Commit message: Preserve M5B-E1 integrated RF2M evaluation baseline
Other:
- note added: "M5B-E1 / integrated evaluation PCB / NOT RELEASED / hardware tests NOT_RUN"
- note added: "M5B-E1: REVIEW / ALL hardware measurements NOT RUN / no ordering or manufacture."
- note removed: "M5A-R4: REVIEW / ALL hardware measurements NOT RUN / no ordering or manufacture."
- note removed: "M5A-R4: hardware measurements NOT_RUN; source/reference and simplification in R4 documents."

Commit message: Implement M5B-E3 standard JLCPCB RF2M evaluation board
Recalculate and implement 1.6 mm / 1 oz RF geometry, power copper, thermal vias, connector holes and manufacturing legend. Preserve electrical functions and population variants. Add native-geometry DFM, regression checks and fresh native/fabrication review archives. CAD milestone only; no manufacturing or operational release.
Parts:
- C507, C508: footprint Capacitor_SMD:C_0603_1608Metric -> ARDF_2M:C_0603_1608Metric_E3
- R515: footprint Resistor_SMD:R_0603_1608Metric -> ARDF_2M:R_0603_1608Metric_E3
- TP501, TP502, TP503: footprint TestPoint:TestPoint_Pad_D1.0mm -> ARDF_2M:TestPoint_Pad_D1.0mm_E3
Other:
- note added: "M5B-E3 / integrated evaluation PCB / NOT RELEASED / hardware tests NOT_RUN"
- note added: "M5B-E3: REVIEW / ALL hardware measurements NOT RUN / no ordering or manufacture."
- note removed: "M5B-E1 / integrated evaluation PCB / NOT RELEASED / hardware tests NOT_RUN"
- note removed: "M5B-E1: REVIEW / ALL hardware measurements NOT RUN / no ordering or manufacture."

Commit message: Implement M5B-E4 thermal candidate with source-joint assembly hold
Other:
- note added: "M5B-E4 / integrated evaluation PCB / NOT RELEASED / hardware tests NOT_RUN"
- note added: "M5B-E4: REVIEW / ALL hardware measurements NOT RUN / no ordering or manufacture."
- note removed: "M5B-E3 / integrated evaluation PCB / NOT RELEASED / hardware tests NOT_RUN"
- note removed: "M5B-E3: REVIEW / ALL hardware measurements NOT RUN / no ordering or manufacture."

Commit message: Implement M5B-E4R1 source-joint prototype candidate
Replace source mask islands with a controlled open-via hybrid and native-derived local stencil. Preserve standard JLCPCB and RF circuitry. Add assembly qualification, thermal convergence and adverse sensitivities, native DFM/mutation checks and fresh review exports. Conservative 110 C target is missed; 125 C physical gate stays open. No acceptance tag or manufacturing authorization.
Other:
- note added: "M5B-E4R1R1R1 / integrated evaluation PCB / NOT RELEASED / hardware tests NOT_RUN"
- note added: "M5B-E4R1R1R1: REVIEW / ALL hardware measurements NOT RUN / no ordering or manufacture."
- note removed: "M5B-E4 / integrated evaluation PCB / NOT RELEASED / hardware tests NOT_RUN"
- note removed: "M5B-E4: REVIEW / ALL hardware measurements NOT RUN / no ordering or manufacture."

Commit message: M5B-E5: compact RF2M to the shared 150x110 mm platform
Other:
- note added: "M5B-E5R1R1 / integrated evaluation PCB / NOT RELEASED / hardware tests NOT_RUN"
- note added: "M5B-E5R1R1: REVIEW / ALL hardware measurements NOT RUN / no ordering or manufacture."
- note removed: "M5B-E4R1R1R1 / integrated evaluation PCB / NOT RELEASED / hardware tests NOT_RUN"
- note removed: "M5B-E4R1R1R1: REVIEW / ALL hardware measurements NOT RUN / no ordering or manufacture."

Commit message: M5B-E6R2: Implement carrier-keyed RF2M and unified cooling
Other:
- note added: "M5B-E6R2 / integrated evaluation PCB / NOT RELEASED / hardware tests NOT_RUN"
- note added: "M5B-E6R2: REVIEW / ALL hardware measurements NOT RUN / no ordering or manufacture."
- note removed: "M5B-E5R1R1 / integrated evaluation PCB / NOT RELEASED / hardware tests NOT_RUN"
- note removed: "M5B-E5R1R1: REVIEW / ALL hardware measurements NOT RUN / no ordering or manufacture."
