File: hardware/2m/06_source_driver_bias.kicad_sch (KiCad schematic)
At the start: 25 parts, among them Q501 PD54008L-E, Q502 2N7002, U501 PHA-1+

Commit message: Preserve M5B-E1 integrated RF2M evaluation baseline
Parts:
- C601: Engineering_Note VHF C0G; Q/SRF and exact MPN OPEN. -> VHF C0G; Q/SRF and exact MPN OPEN. Selected Yageo C0G50V;ex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; MPN OPEN: 0603 C0G50V 100p -> CC0603JRNPO9BN101
- C602: Engineering_Note MMIC output DC block; connects to ST interstage derivative,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 -> Existing1nF MMIC output DC block;R650 liftable link now iso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
- C611, C614: Engineering_Note VHF C0G; Q/SRF and exact MPN OPEN. -> VHF C0G; Q/SRF and exact MPN OPEN. Selected Yageo C0G50V;ex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; MPN OPEN: 0603 C0G50V 8.2p -> CC0603CRNPO9BN8R2
- C612, C613: Engineering_Note VHF C0G; Q/SRF and exact MPN OPEN. -> VHF C0G; Q/SRF and exact MPN OPEN. Selected Yageo C0G50V;ex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; MPN OPEN: 0603 C0G50V 33p -> CC0603JRNPO9BN330
- L604: value 180n -> 150n; footprint Inductor_SMD:L_0603_1608Metric -> ARDF_2M:Coilcraft_1812SMS_Doc184; Engineering_Note Low-power RF path only.56n Q>=38@200MHz SRF2.6GHz Imax770mA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 -> M5B corrects actualMMIC DC bias loss:originalMurata180n max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; MPN LQW18ANR18G80D -> 1812SMS-R15JLC
- L606: footprint (none) -> ARDF_2M:Coilcraft_1812SMS_Doc184; Engineering_Note ST Fig13 L2 final gate feed33nH retained; participates in i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 -> RetainedST33nH feed;M5B exactDoc184-2 staggered land/curren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
- R602: value 17.8 -> 71.5; Engineering_Note 3dB pi-pad candidate17.6/292.4 theoretical, rounded17.8/287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 -> Initial10dB50ohm pi pad;after one integrated calibration6/8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; MPN RC0603FR-0717R8L -> RC0603FR-0771R5L
- R603, R604: value 287 -> 96.5; Engineering_Note (none) -> Initial10dB50ohm pi pad;after one integrated calibration6/8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; MPN RC0603FR-07287RL -> RC0603FR-0796R5L
- TP601: footprint TestPoint:TestPoint_Pad_D1.0mm -> ARDF_2M:Probe_Pad_0p6
Connections:
- net MMIC_AC renamed MMIC_COUPLED
- net VDRV_RF renamed VDRV_MMIC
Other:
- note added: "M5B-E1 / integrated evaluation PCB / NOT RELEASED / hardware tests NOT_RUN"
- note added: "M5B-E1: REVIEW / ALL hardware measurements NOT RUN / no ordering or manufacture."
- note removed: "M5A-R4: REVIEW / ALL hardware measurements NOT RUN / no ordering or manufacture."
- note removed: "M5A-R4: hardware measurements NOT_RUN; source/reference and simplification in R4 documents."

Commit message: Implement M5B-E3 standard JLCPCB RF2M evaluation board
Recalculate and implement 1.6 mm / 1 oz RF geometry, power copper, thermal vias, connector holes and manufacturing legend. Preserve electrical functions and population variants. Add native-geometry DFM, regression checks and fresh native/fabrication review archives. CAD milestone only; no manufacturing or operational release.
Parts:
- C601, C602, C603, C604, C607, C611, C612, C613, C614, C615: footprint Capacitor_SMD:C_0603_1608Metric -> ARDF_2M:C_0603_1608Metric_E3
- D501: footprint Diode_SMD:D_SOD-123F -> ARDF_2M:D_SOD-123F_E3
- L611, L612, L613: footprint Inductor_SMD:L_0603_1608Metric -> ARDF_2M:L_0603_1608Metric_E3
- Q502: footprint Package_TO_SOT_SMD:SOT-23 -> ARDF_2M:SOT-23_E3
- R602, R603, R604, R606: footprint Resistor_SMD:R_0603_1608Metric -> ARDF_2M:R_0603_1608Metric_E3
- RV501: footprint Potentiometer_THT:Potentiometer_Bourns_3296W_Vertical -> ARDF_2M:Potentiometer_Bourns_3296W_Vertical_E3
Other:
- note added: "M5B-E3 / integrated evaluation PCB / NOT RELEASED / hardware tests NOT_RUN"
- note added: "M5B-E3: REVIEW / ALL hardware measurements NOT RUN / no ordering or manufacture."
- note removed: "M5B-E1 / integrated evaluation PCB / NOT RELEASED / hardware tests NOT_RUN"
- note removed: "M5B-E1: REVIEW / ALL hardware measurements NOT RUN / no ordering or manufacture."

Commit message: Implement M5B-E4 thermal candidate with source-joint assembly hold
Other:
- note added: "M5B-E4 / integrated evaluation PCB / NOT RELEASED / hardware tests NOT_RUN"
- note added: "M5B-E4: REVIEW / ALL hardware measurements NOT RUN / no ordering or manufacture."
- note removed: "M5B-E3 / integrated evaluation PCB / NOT RELEASED / hardware tests NOT_RUN"
- note removed: "M5B-E3: REVIEW / ALL hardware measurements NOT RUN / no ordering or manufacture."

Commit message: Implement M5B-E4R1 source-joint prototype candidate
Replace source mask islands with a controlled open-via hybrid and native-derived local stencil. Preserve standard JLCPCB and RF circuitry. Add assembly qualification, thermal convergence and adverse sensitivities, native DFM/mutation checks and fresh review exports. Conservative 110 C target is missed; 125 C physical gate stays open. No acceptance tag or manufacturing authorization.
Other:
- note added: "M5B-E4R1R1R1 / integrated evaluation PCB / NOT RELEASED / hardware tests NOT_RUN"
- note added: "M5B-E4R1R1R1: REVIEW / ALL hardware measurements NOT RUN / no ordering or manufacture."
- note removed: "M5B-E4 / integrated evaluation PCB / NOT RELEASED / hardware tests NOT_RUN"
- note removed: "M5B-E4: REVIEW / ALL hardware measurements NOT RUN / no ordering or manufacture."

Commit message: M5B-E5: compact RF2M to the shared 150x110 mm platform
Other:
- note added: "M5B-E5R1R1 / integrated evaluation PCB / NOT RELEASED / hardware tests NOT_RUN"
- note added: "M5B-E5R1R1: REVIEW / ALL hardware measurements NOT RUN / no ordering or manufacture."
- note removed: "M5B-E4R1R1R1 / integrated evaluation PCB / NOT RELEASED / hardware tests NOT_RUN"
- note removed: "M5B-E4R1R1R1: REVIEW / ALL hardware measurements NOT RUN / no ordering or manufacture."

Commit message: M5B-E6R2: Implement carrier-keyed RF2M and unified cooling
Other:
- note added: "M5B-E6R2 / integrated evaluation PCB / NOT RELEASED / hardware tests NOT_RUN"
- note added: "M5B-E6R2: REVIEW / ALL hardware measurements NOT RUN / no ordering or manufacture."
- note removed: "M5B-E5R1R1 / integrated evaluation PCB / NOT RELEASED / hardware tests NOT_RUN"
- note removed: "M5B-E5R1R1: REVIEW / ALL hardware measurements NOT RUN / no ordering or manufacture."
