File: hardware/2m/10_enable_detail.kicad_sch (KiCad schematic)
At the start: 13 parts, among them U205 74HC21D,653, U206 74HC11D,653, U305 TPS22919DCKR, U601 SN74LVC1G125DBVR

Commit message: Preserve M5B-E1 integrated RF2M evaluation baseline
Parts:
- U305: value TPS22919DCKR -> TPS22810DBVR; footprint Package_TO_SOT_SMD:SOT-363_SC-70-6 -> Package_TO_SOT_SMD:SOT-23-6; symbol ARDF_2M:TPS22919 -> ARDF_2M:TPS22810_DBV; Engineering_Note TI physical1VIN2GND3ON4NC5QOD6VOUT.5V switch only, never9V/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 -> TI DBV1VIN2GND3EN4CT5QOD6OUT.2.7-18V recommended,20Vabs. CT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; MPN TPS22919DCKR -> TPS22810DBVR
Other:
- note added: "M5B-E1 / integrated evaluation PCB / NOT RELEASED / hardware tests NOT_RUN"
- note added: "M5B-E1: REVIEW / ALL hardware measurements NOT RUN / no ordering or manufacture."
- note removed: "M5A-R4: REVIEW / ALL hardware measurements NOT RUN / no ordering or manufacture."
- note removed: "One integrated transmitter, no separate coupon.9V fixed converter, separate filtered5V driver. TPS22919 replaces discrete driver-switch network. Source gate delays only turn-on; fail-off uses direct inhibit and rail isolation. RC timings, analog trip latency and real RF silence remain physical acceptance gates."

Commit message: Implement M5B-E3 standard JLCPCB RF2M evaluation board
Recalculate and implement 1.6 mm / 1 oz RF geometry, power copper, thermal vias, connector holes and manufacturing legend. Preserve electrical functions and population variants. Add native-geometry DFM, regression checks and fresh native/fabrication review archives. CAD milestone only; no manufacturing or operational release.
Parts:
- C931, C940, C941: footprint Capacitor_SMD:C_0603_1608Metric -> ARDF_2M:C_0603_1608Metric_E3
- D930: footprint Diode_SMD:D_SOD-323 -> ARDF_2M:D_SOD-323_E3
- R930, R931, R932, R940: footprint Resistor_SMD:R_0603_1608Metric -> ARDF_2M:R_0603_1608Metric_E3
- TP940: footprint TestPoint:TestPoint_Pad_D1.0mm -> ARDF_2M:TestPoint_Pad_D1.0mm_E3
- U205, U206: footprint Package_SO:SOIC-14_3.9x8.7mm_P1.27mm -> ARDF_2M:SOIC-14_3.9x8.7mm_P1.27mm_E3
- U305: footprint Package_TO_SOT_SMD:SOT-23-6 -> ARDF_2M:SOT-23-6_E3
- U601: footprint Package_TO_SOT_SMD:SOT-23-5 -> ARDF_2M:SOT-23-5_E3
Other:
- note added: "M5B-E3 / integrated evaluation PCB / NOT RELEASED / hardware tests NOT_RUN"
- note added: "M5B-E3: REVIEW / ALL hardware measurements NOT RUN / no ordering or manufacture."
- note removed: "M5B-E1 / integrated evaluation PCB / NOT RELEASED / hardware tests NOT_RUN"
- note removed: "M5B-E1: REVIEW / ALL hardware measurements NOT RUN / no ordering or manufacture."

Commit message: Implement M5B-E4 thermal candidate with source-joint assembly hold
Other:
- note added: "M5B-E4 / integrated evaluation PCB / NOT RELEASED / hardware tests NOT_RUN"
- note added: "M5B-E4: REVIEW / ALL hardware measurements NOT RUN / no ordering or manufacture."
- note removed: "M5B-E3 / integrated evaluation PCB / NOT RELEASED / hardware tests NOT_RUN"
- note removed: "M5B-E3: REVIEW / ALL hardware measurements NOT RUN / no ordering or manufacture."

Commit message: Implement M5B-E4R1 source-joint prototype candidate
Replace source mask islands with a controlled open-via hybrid and native-derived local stencil. Preserve standard JLCPCB and RF circuitry. Add assembly qualification, thermal convergence and adverse sensitivities, native DFM/mutation checks and fresh review exports. Conservative 110 C target is missed; 125 C physical gate stays open. No acceptance tag or manufacturing authorization.
Other:
- note added: "M5B-E4R1R1R1 / integrated evaluation PCB / NOT RELEASED / hardware tests NOT_RUN"
- note added: "M5B-E4R1R1R1: REVIEW / ALL hardware measurements NOT RUN / no ordering or manufacture."
- note removed: "M5B-E4 / integrated evaluation PCB / NOT RELEASED / hardware tests NOT_RUN"
- note removed: "M5B-E4: REVIEW / ALL hardware measurements NOT RUN / no ordering or manufacture."

Commit message: M5B-E5: compact RF2M to the shared 150x110 mm platform
Other:
- note added: "M5B-E5R1R1 / integrated evaluation PCB / NOT RELEASED / hardware tests NOT_RUN"
- note added: "M5B-E5R1R1: REVIEW / ALL hardware measurements NOT RUN / no ordering or manufacture."
- note removed: "M5B-E4R1R1R1 / integrated evaluation PCB / NOT RELEASED / hardware tests NOT_RUN"
- note removed: "M5B-E4R1R1R1: REVIEW / ALL hardware measurements NOT RUN / no ordering or manufacture."

Commit message: M5B-E6R2: Implement carrier-keyed RF2M and unified cooling
Connections:
- net NORMAL_PERMIT: no longer U305.3 (EN)
- net NORMAL_OFF renamed CLOCK_OFF
- new net DRIVER_ON: U305.3 (EN)
Other:
- note added: "M5B-E6R2 / integrated evaluation PCB / NOT RELEASED / hardware tests NOT_RUN"
- note added: "M5B-E6R2: REVIEW / ALL hardware measurements NOT RUN / no ordering or manufacture."
- note removed: "M5B-E5R1R1 / integrated evaluation PCB / NOT RELEASED / hardware tests NOT_RUN"
- note removed: "M5B-E5R1R1: REVIEW / ALL hardware measurements NOT RUN / no ordering or manufacture."
