File: hardware/2m/11_external_contract.kicad_sch (KiCad schematic)
At the start: 0 parts

Commit message: Preserve M5A-R4 economical VHF electrical review baseline
Other:
- note added: "11 External supplies and integrated commissioning"
- note added: "M5A-R4: REVIEW / ALL hardware measurements NOT RUN / no ordering or manufacture."
- note added: "R4 MPN/landing blockers are explicit. No PCB manufacturing release. All physical RF/AM/thermal tests NOT_RUN. The measured antenna gain sets ERP calibration;1dB reserve is optional engineering headroom, NOT an IARU rule. Controller: R4 IDs,144MHz direct clocks,2S fixed9V /4S9Vfull7.5Vreduced;AF/DC calibrated separately; keep20pin pinout."
- note removed: "11 External supply declarations and qualification boundary"
- note removed: "M5A-R3: REVIEW / ALL hardware measurements NOT RUN / no ordering or manufacture."
- note removed: "No PCB is released: exact final manufacturer/lot, some magnetic/choke/trimmer geometry and RF source coupling remain OPEN. No physical measurements exist. See M5A_R3_REVIEW_DECISION.md. PWR_FLAG is an ERC declaration, not a safety approval."
- title: 11 External supply declarations and qualification boundary -> 11 External supplies and integrated commissioning

Commit message: Preserve M5B-E1 integrated RF2M evaluation baseline
Other:
- note added: "M5B-E1 / integrated evaluation PCB / NOT RELEASED / hardware tests NOT_RUN"
- note added: "M5B-E1: REVIEW / ALL hardware measurements NOT RUN / no ordering or manufacture."
- note removed: "M5A-R4: REVIEW / ALL hardware measurements NOT RUN / no ordering or manufacture."
- note removed: "R4 MPN/landing blockers are explicit. No PCB manufacturing release. All physical RF/AM/thermal tests NOT_RUN. The measured antenna gain sets ERP calibration;1dB reserve is optional engineering headroom, NOT an IARU rule. Controller: R4 IDs,144MHz direct clocks,2S fixed9V /4S9Vfull7.5Vreduced;AF/DC calibrated separately; keep20pin pinout."

Commit message: Implement M5B-E3 standard JLCPCB RF2M evaluation board
Recalculate and implement 1.6 mm / 1 oz RF geometry, power copper, thermal vias, connector holes and manufacturing legend. Preserve electrical functions and population variants. Add native-geometry DFM, regression checks and fresh native/fabrication review archives. CAD milestone only; no manufacturing or operational release.
Other:
- note added: "M5B-E3 / integrated evaluation PCB / NOT RELEASED / hardware tests NOT_RUN"
- note added: "M5B-E3: REVIEW / ALL hardware measurements NOT RUN / no ordering or manufacture."
- note removed: "M5B-E1 / integrated evaluation PCB / NOT RELEASED / hardware tests NOT_RUN"
- note removed: "M5B-E1: REVIEW / ALL hardware measurements NOT RUN / no ordering or manufacture."

Commit message: Implement M5B-E4 thermal candidate with source-joint assembly hold
Other:
- note added: "M5B-E4 / integrated evaluation PCB / NOT RELEASED / hardware tests NOT_RUN"
- note added: "M5B-E4: REVIEW / ALL hardware measurements NOT RUN / no ordering or manufacture."
- note removed: "M5B-E3 / integrated evaluation PCB / NOT RELEASED / hardware tests NOT_RUN"
- note removed: "M5B-E3: REVIEW / ALL hardware measurements NOT RUN / no ordering or manufacture."

Commit message: Implement M5B-E4R1 source-joint prototype candidate
Replace source mask islands with a controlled open-via hybrid and native-derived local stencil. Preserve standard JLCPCB and RF circuitry. Add assembly qualification, thermal convergence and adverse sensitivities, native DFM/mutation checks and fresh review exports. Conservative 110 C target is missed; 125 C physical gate stays open. No acceptance tag or manufacturing authorization.
Other:
- note added: "M5B-E4R1R1R1 / integrated evaluation PCB / NOT RELEASED / hardware tests NOT_RUN"
- note added: "M5B-E4R1R1R1: REVIEW / ALL hardware measurements NOT RUN / no ordering or manufacture."
- note removed: "M5B-E4 / integrated evaluation PCB / NOT RELEASED / hardware tests NOT_RUN"
- note removed: "M5B-E4: REVIEW / ALL hardware measurements NOT RUN / no ordering or manufacture."

Commit message: M5B-E5: compact RF2M to the shared 150x110 mm platform
Other:
- note added: "M5B-E5R1R1 / integrated evaluation PCB / NOT RELEASED / hardware tests NOT_RUN"
- note added: "M5B-E5R1R1: REVIEW / ALL hardware measurements NOT RUN / no ordering or manufacture."
- note removed: "M5B-E4R1R1R1 / integrated evaluation PCB / NOT RELEASED / hardware tests NOT_RUN"
- note removed: "M5B-E4R1R1R1: REVIEW / ALL hardware measurements NOT RUN / no ordering or manufacture."

Commit message: M5B-E6R2: Implement carrier-keyed RF2M and unified cooling
Other:
- note added: "M5B-E6R2 / integrated evaluation PCB / NOT RELEASED / hardware tests NOT_RUN"
- note added: "M5B-E6R2: REVIEW / ALL hardware measurements NOT RUN / no ordering or manufacture."
- note removed: "M5B-E5R1R1 / integrated evaluation PCB / NOT RELEASED / hardware tests NOT_RUN"
- note removed: "M5B-E5R1R1: REVIEW / ALL hardware measurements NOT RUN / no ordering or manufacture."
