File: hardware/controller/01_power.kicad_sch (KiCad schematic)
At the start: 18 parts, among them J1 PACK / GND / ID, U1 AP63203WU-7

Commit message: M6-C1R1: protect pack identity input and review USB ESD topology
Parts:
- R3: value 10k -> 27k; Engineering_Note Yageo RC0603 1%, 0.1W -> 1%,0.1W; pack-derived ID excitation, no V3V3 connection; MPN RC0603FR-0710KL -> RC0603FR-0727KL
Connections:
- net V3V3: no longer R3.1
- new net PACK_ID_EXC: R3.1
Other:
- note added: "M6-C1R1 candidate: REVIEW / ALL hardware measurements NOT RUN / no ordering or manufacture."
- note removed: "M6-C1 candidate: REVIEW / ALL hardware measurements NOT RUN / no ordering or manufacture."
