File: hardware/controller/01_power_2.kicad_sch (KiCad schematic)
At the start: 5 parts, among them Q1 MMBT3904

Commit message: M6-C1R1: protect pack identity input and review USB ESD topology
Parts:
- added D22: BAS116 ID excitation isolation, ARDF_CTL:SOT-23_CTL, symbol ARDF_CTL:M6_D22
- added D23: BAT54H negative ID clamp, ARDF_CTL:D_SOD-123F_CTL, symbol ARDF_CTL:D_Schottky
- added R19: 100k, ARDF_CTL:R_0603_1608Metric_CTL, symbol ARDF_CTL:R
- added R8: 180k, ARDF_CTL:R_0603_1608Metric_CTL, symbol ARDF_CTL:R
- added R9: 33k, ARDF_CTL:R_0603_1608Metric_CTL, symbol ARDF_CTL:R
Connections:
- net GND: now also D23.2 (A), R19.2, R9.2
- net PACK_PROT: now also D22.1 (1_A)
- new net PACK_ID_ADC: R19.1
- new net PACK_ID_EXC: D22.3 (3_K)
- new net PACK_ID_RAW: R8.1
- new net PACK_ID_SAFE: D23.1 (K), R8.2, R9.1
- no-connect marks 0 -> 1
Other:
- note added: "M6-C1R1 candidate: REVIEW / ALL hardware measurements NOT RUN / no ordering or manufacture."
- note removed: "M6-C1 candidate: REVIEW / ALL hardware measurements NOT RUN / no ordering or manufacture."
- moved on the sheet: Q1, R4, R5, R6, R7
