File: hardware/controller/04_RTC_analog.kicad_sch (KiCad schematic)
At the start: 17 parts, among them U20 RV-3032-C7 2.5ppm, U21 TMUX1511PWR

Commit message: M6-C1R1: protect pack identity input and review USB ESD topology
Parts:
- U21: Engineering_Note Powered-off protected four analog channels. Signals remain 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 -> Powered-off protected four analog channels. Signal limit3.6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
Connections:
- net PACK_ID_RAW renamed PACK_ID_SAFE
Other:
- note added: "M6-C1R1 candidate: REVIEW / ALL hardware measurements NOT RUN / no ordering or manufacture."
- note removed: "M6-C1 candidate: REVIEW / ALL hardware measurements NOT RUN / no ordering or manufacture."
