File: hardware/controller/05_static_safety_2.kicad_sch (KiCad schematic)
At the start: 18 parts, among them U32 SN74LVC1G04DBVR, U33 SN74LVC1G10DBVR, U34 SN74LVC2G04DCKR, U35 SN74LVC00APWR, U36 SN74LVC1G04DBVR, U37 SN74LVC08APWR

Commit message: M6-C1R1: protect pack identity input and review USB ESD topology
Other:
- note added: "M6-C1R1 candidate: REVIEW / ALL hardware measurements NOT RUN / no ordering or manufacture."
- note removed: "M6-C1 candidate: REVIEW / ALL hardware measurements NOT RUN / no ordering or manufacture."
