File: hardware/controller/CTRL.kicad_pcb (KiCad board)
At the start: 2 copper layers, 100 x 100 mm, 200 parts, among them J1 PACK / GND / ID, J2 USB-C native USB2, J3 UART recovery / GND, J4 RF80 keyed controller link, J5 RF2M keyed controller link, J7 LoRa antenna U.FL, Q1 MMBT3904, Q2 MMBT3904 VBUS sense, SW1 RESET, SW2 BOOT, SW3 START, SW4 STOP / hold reset, U1 AP63203WU-7, U10 ESP32-S3-WROOM-1-N4, U2 TPS2553DBVR, U20 RV-3032-C7 2.5ppm, U21 TMUX1511PWR, U3 USBLC6-2SC6, U30 SN74HC595PWR, U31 SN74HC595PWR, U32 SN74LVC1G04DBVR, U33 SN74LVC1G10DBVR, U34 SN74LVC2G04DCKR, U35 SN74LVC00APWR, U36 SN74LVC1G04DBVR, U37 SN74LVC08APWR, U4 TLV803EA30DBZR, U40 TPS22918DBVR, U41 SN74LVC244APWR, U42 SN74LVC125APWR, U43 TCA9517DR, U50 TPS22918DBVR, U51 SN74LVC244APWR, U52 SN74LVC125APWR, U53 TCA9517DR, U60 SN74LVC2G17DCKR, U70 Silicontra SX1262ZTR8-GC

Commit message: M6-C1R1: protect pack identity input and review USB ESD topology
Parts:
- added D22: BAS116 ID excitation isolation, ARDF_CTL:SOT-23_CTL, B.Cu at (41.0, 99.0)
- added D23: BAT54H negative ID clamp, ARDF_CTL:D_SOD-123F_CTL, B.Cu at (54.0, 116.5)
- added R19: 100k, ARDF_CTL:R_0603_1608Metric_CTL, B.Cu at (89.0, 54.5)
- added R8: 180k, ARDF_CTL:R_0603_1608Metric_CTL, B.Cu at (45.0, 115.0)
- added R9: 33k, ARDF_CTL:R_0603_1608Metric_CTL, B.Cu at (49.0, 116.5)
- R3: value 10k -> 27k; moved to B.Cu
- moved R3 54.1 mm to (42.0, 104.0), turned to 90 degrees
Connections:
- C25 pad 1: PACK_ID_RAW -> PACK_ID_SAFE
- R3 pad 1: V3V3 -> PACK_ID_EXC
- U21 pad 5: PACK_ID_RAW -> PACK_ID_SAFE
Routing:
- net PACK_ID_SAFE: track 0.00 -> 95.1 mm, vias 0 -> 5
- net PACK_ID_RAW: track 81.4 -> 20.5 mm, vias 1 -> 0
- net PACK_ID_ADC: track 37.2 -> 54.9 mm, vias 2 -> 4
- net PACK_ID_EXC: track 0.00 -> 10.1 mm, vias 0 -> 2
- net PACK_PROT: track 125.0 -> 128.4 mm, vias 4 -> 5
- net V3V3: track 461.5 -> 459.7 mm
Other:
- board text added: "ARDF-TX C1R1"
- board text removed: "ARDF-TX M6-C1"

Commit message: M6-L1: close dual-band Silicontra footprint and RF feed review
Verify TR4/TR8 supplier aliases and all 22 nominal module terminals; retain
the common RF signal feed and Hirose lands. Remove a local ground-fill
intrusion in the full U.FL underbody keep-out and correct the module body
outline and unused DIO3 label.

Add explicit no-radio/433/868 assembly records, fail-disabled band/policy
fixtures, native-geometry mutations, tolerance RF calculations and fresh
standard-JLCPCB fabrication/assembly exports with source-bound manifests.

KiCad 10.0.6 ERC/DRC warnings/errors, unrouted and parity all zero. Preserve
704 pad assertions, 36 RF pins, 4096 enable cases, R1 protection/DFM tests,
46 host tests and strict C11 fixture. Physical qualification NOT_RUN.
Independent manufacturing review candidate only; no acceptance tag.
Parts:
- U70: value Silicontra SX1262ZTR8-GC -> Silicontra SX1262TR8-GC
Other:
- board text added: "ARDF-TX L1"
- board text removed: "ARDF-TX C1R1"
Changed lines of the file:
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@@
 		(title "ARDF-TX UNIVERSAL CONTROLLER")
 		(date "2026-10-18")
-		(rev "M6-C1R1 CANDIDATE")
+		(rev "M6-L1 CANDIDATE")
 		(company "ARDF-TX")
 		(comment 1 "ENGINEERING REVIEW ONLY / PHYSICAL TESTS NOT_RUN")
@@
 			)
 		)
-		(property "Population" "LORA_OPTION_OPEN"
+		(property "Population" "LORA_OPTION"
 			(at 0 0 0)
 			(layer "F.SilkS")
@@
 			)
 		)
-		(property "Population" "LORA_OPTION_OPEN"
+		(property "Population" "LORA_OPTION"
 			(at 0 0 90)
 			(layer "F.SilkS")
@@
 			)
 		)
-		(property "Population" "LORA_OPTION_OPEN"
+		(property "Population" "LORA_OPTION"
 			(at 0 0 0)
 			(layer "F.SilkS")
@@
 			)
 		)
-		(property "Population" "LORA_OPTION_OPEN"
+		(property "Population" "LORA_OPTION"
 			(at 0 0 90)
 			(layer "F.SilkS")
@@
 			)
 		)
-		(property "Population" "LORA_OPTION_OPEN"
+		(property "Population" "LORA_OPTION"
 			(at 0 0 0)
 			(layer "F.SilkS")
@@
 			)
 		)
-		(property "Engineering_Note" "Pin1 signal; duplicated pin2 ground. Underbody copper keepout preserved, exposed-mask-only rectangle omitted. External868MHz antenna; optional module footprint review OPEN."
+		(property "Engineering_Note" "M6-L1: Hirose U.FL-R-SMT-1(10), available cut tape MOQ1. Same antenna feed433/868; choose band-correct external antenna. Nominal copper lands retained; see manufacturer pattern/assembly audit."
 			(at 0 0 0)
 			(layer "F.SilkS")
@@
 			)
 		)
-		(property "Value" "Silicontra SX1262ZTR8-GC"
+		(property "Value" "Silicontra SX1262TR8-GC"
 			(at 0 9.35 0)
 			(layer "F.Fab")
@@
 			)
 		)
-		(property "MPN" "SX1262ZTR8-GC"
+		(property "MPN" "SX1262TR8-GC"
 			(at 0 0 0)
 			(layer "F.SilkS")
@@
 			)
 		)
-		(property "Population" "LORA_OPTION_OPEN"
+		(property "Population" "LORA_OPTION"
 			(at 0 0 0)
 			(layer "F.SilkS")
@@
 			)
 		)
-		(property "Engineering_Note" "OPTIONAL DNP: manufacturer ZTR8 vs distributor TR8 suffix not confirmed. Manufacturer dimension drawing lacks tolerances and ambiguous 1.12mm callout; footprint qualification OPEN. Do not populate without review."
+		(property "Engineering_Note" "M6-L1: TR4/ZTR4 and TR8/ZTR8 supplier-linked manufacturer documents agree on22pin15x15 package. Common footprint; select trusted433/868 assembly record and matching antenna. DIO3 pin8 is optional IO, unused here. Incoming identity/fit and RF qualification NOT_RUN."
 			(at 0 0 0)
 			(layer "F.SilkS")
@@
 		)
 		(fp_rect
-			(start -7.5 -8.35)
-			(end 7.5 8.35)
+			(start -7.5 -7.5)
+			(end 7.5 7.5)
 			(stroke
 				(width 0.1)
@@
 			(size 0.8 2.2)
 			(layers "F.Cu" "F.Mask" "F.Paste")
-			(net "unconnected-(U70-8_IO-Pad8)")
+			(net "unconnected-(U70-8_DIO3-Pad8)")
 		)
 		(pad "9" smd rect
@@
 		)
 	)
-	(gr_text "ARDF-TX C1R1"
+	(gr_text "ARDF-TX L1"
 		(at 88 22.5 0)
 		(layer "F.SilkS")
@@
 			(tracks not_allowed)
 			(vias not_allowed)
-			(pads not_allowed)
+			(pads allowed)
 			(copperpour not_allowed)
 			(footprints allowed)
@@
 		(polygon
 			(pts
-				(xy 100.515 27.55) (xy 98.425 27.55) (xy 98.425 29.45) (xy 100.515 29.45)
+				(xy 98.315 27.55) (xy 100.515 27.55) (xy 100.515 29.45) (xy 98.315 29.45)
 			)
 		)

Commit message: M6-L2 — External antenna, FoxPro2 interface and GPIO expansion
Parts:
- added C80: 100n, ARDF_CTL:C_0603_1608Metric_CTL, F.Cu at (48.5, 25.0)
- added C81: 100n, ARDF_CTL:C_0603_1608Metric_CTL, B.Cu at (86.5, 43.5)
- added C82: 100n, ARDF_CTL:C_0603_1608Metric_CTL, B.Cu at (96.2, 52.2)
- added C83: 100n, ARDF_CTL:C_0603_1608Metric_CTL, F.Cu at (61.5, 37.8)
- added C84: 10n, ARDF_CTL:C_0603_1608Metric_CTL, B.Cu at (61.2, 26.5)
- added D80: PESD1IVN24-A bidirectional TVS, ARDF_CTL:D_SOD-323_L2, F.Cu at (86.0, 22.5)
- added D81: BAS316 negative collector clamp, ARDF_CTL:D_SOD-323_L2, B.Cu at (54.5, 22.5)
- added D82: BZX84-C12 gate clamp, ARDF_CTL:SOT-23_CTL, F.Cu at (67.0, 26.0)
- added D83: PESD1IVN24-A bidirectional TVS, ARDF_CTL:D_SOD-323_L2, F.Cu at (93.0, 23.0)
- added D84: PESD1IVN24-A bidirectional TVS, ARDF_CTL:D_SOD-323_L2, F.Cu at (90.0, 23.0)
- added J8: FOXPRO / G-D-V UNAVAILABLE, ARDF_CTL:JST_PH_B3B-PH-K_1x03_P2.00mm_Vertical_L2, B.Cu at (83.5, 26.0)
- added J9: GPIO / 3V3 ONLY / 10mA, ARDF_CTL:PinHeader_2x05_P2.54mm_Vertical_L2, B.Cu at (36.0, 25.5)
- added JP1: GPIO3 SERVICE ONLY / OPEN, ARDF_CTL:SolderJumper-2_P1.3mm_Open_Pad1.0x1.5mm_L2, B.Cu at (40.0, 39.0)
- added JP3: GPIO46 SERVICE ONLY / OPEN, ARDF_CTL:SolderJumper-2_P1.3mm_Open_Pad1.0x1.5mm_L2, B.Cu at (46.0, 43.0)
- added Q80: BSS138BK TX open-drain, ARDF_CTL:SOT-23_CTL, B.Cu at (64.0, 24.0)
- added Q81: MMBT3904 hardware inhibit, ARDF_CTL:SOT-23_CTL, B.Cu at (72.5, 23.0)
- added Q82: BSS138BK isolated-gate RX, ARDF_CTL:SOT-23_CTL, B.Cu at (68.0, 23.5)
- added R300: 0, ARDF_CTL:R_0603_1608Metric_CTL, F.Cu at (64.5, 33.9)
- added R301: 0, ARDF_CTL:R_0603_1608Metric_CTL, F.Cu at (68.0, 34.8)
- added R302: 0, ARDF_CTL:R_0603_1608Metric_CTL, B.Cu at (74.0, 32.5)
- added R303: 0, ARDF_CTL:R_0603_1608Metric_CTL, B.Cu at (67.0, 33.8)
- added R304: 680, ARDF_CTL:R_2512_6332Metric_L2, B.Cu at (76.5, 27.0)
- added R305: 1k, ARDF_CTL:R_0603_1608Metric_CTL, B.Cu at (78.5, 31.0)
- added R306: 4.7k, ARDF_CTL:R_0603_1608Metric_CTL, B.Cu at (67.0, 27.5)
- added R307: 1k, ARDF_CTL:R_0603_1608Metric_CTL, B.Cu at (64.0, 27.5)
- added R308: 4.7k, ARDF_CTL:R_0603_1608Metric_CTL, B.Cu at (58.5, 23.0)
- added R309: 47k, ARDF_CTL:R_0603_1608Metric_CTL, B.Cu at (75.8, 23.2)
- added R310: 100k, ARDF_CTL:R_0603_1608Metric_CTL, B.Cu at (90.5, 29.5)
- added R311: 160, ARDF_CTL:R_0603_1608Metric_CTL, B.Cu at (91.0, 26.5)
- added R312: 100k, ARDF_CTL:R_0603_1608Metric_CTL, B.Cu at (91.0, 23.0)
- added R313: 0, ARDF_CTL:R_0603_1608Metric_CTL, B.Cu at (93.0, 23.0)
- added R314: 470, ARDF_CTL:R_2512_6332Metric_L2, B.Cu at (88.0, 35.5)
- added R315: 620, ARDF_CTL:R_0603_1608Metric_CTL, B.Cu at (92.0, 31.5)
- added R316: 470, ARDF_CTL:R_2512_6332Metric_L2, B.Cu at (95.5, 37.5)
- added R320: 4.7k, ARDF_CTL:R_0603_1608Metric_CTL, B.Cu at (95.0, 48.5)
- added R321: 4.7k, ARDF_CTL:R_0603_1608Metric_CTL, B.Cu at (94.5, 51.0)
- added R322: 1k, ARDF_CTL:R_0603_1608Metric_CTL, B.Cu at (24.0, 31.0)
- added R323: 1k, ARDF_CTL:R_0603_1608Metric_CTL, B.Cu at (30.0, 36.5)
- added R324: 1k, ARDF_CTL:R_0603_1608Metric_CTL, B.Cu at (39.0, 33.0)
- added R325: 1k, ARDF_CTL:R_0603_1608Metric_CTL, B.Cu at (25.2, 58.2)
- added R326: 1k, ARDF_CTL:R_0603_1608Metric_CTL, B.Cu at (27.0, 32.0)
- added R327: 1k, ARDF_CTL:R_0603_1608Metric_CTL, B.Cu at (30.5, 32.0)
- added R328: 1k, ARDF_CTL:R_0603_1608Metric_CTL, B.Cu at (33.0, 32.0)
- added R329: 1k, ARDF_CTL:R_0603_1608Metric_CTL, B.Cu at (25.0, 67.0)
- added R330: 22, ARDF_CTL:R_2512_6332Metric_L2, B.Cu at (36.0, 35.0)
- added R331: 10k, ARDF_CTL:R_0603_1608Metric_CTL, B.Cu at (67.0, 114.0)
- added TP81: GPIO3 AFTER OPEN LINK, ARDF_CTL:TestPoint_Pad_D1.0mm_CTL, B.Cu at (37.0, 40.2)
- added TP83: GPIO46 AFTER OPEN LINK, ARDF_CTL:TestPoint_Pad_D1.0mm_CTL, B.Cu at (32.0, 59.0)
- added U80: TCA9534APWR / 0x38, ARDF_CTL:TSSOP-16_4.4x5mm_P0.65mm_CTL, B.Cu at (46.0, 24.5)
- added U81: TCA9517DR optional bus buffer, ARDF_CTL:SOIC-8_3.9x4.9mm_P1.27mm_CTL, B.Cu at (89.5, 49.5)
- added U82: LM66100DCKR reverse block, ARDF_CTL:SOT-363_SC-70-6_CTL, F.Cu at (65.0, 37.5)
- U10: value ESP32-S3-WROOM-1-N4 -> ESP32-S3-WROOM-1U-N4; footprint ARDF_CTL:ESP32_S3_WROOM_1_Standard -> ARDF_CTL:ESP32_S3_WROOM_1U_N4_L2
- moved U10 3.15 mm to (50.0, 38.1)
Connections:
- J3 pad 2: UART_TX -> REC_TX
- J3 pad 3: UART_RX -> REC_RX
- U10 pad 15: unconnected-(U10-15_GPIO3-Pad15) -> STRAP3
- U10 pad 16: unconnected-(U10-16_GPIO46-Pad16) -> STRAP46
Routing:
- net EXP_P1: track 0.00 -> 296.1 mm, vias 0 -> 16
- net EXP_VDD: track 0.00 -> 198.7 mm, vias 0 -> 11
- net RTC80_SDA: track 79.6 -> 260.8 mm, vias 4 -> 22
- net RTC80_SCL: track 45.8 -> 189.7 mm, vias 2 -> 17
- net SAFE: track 23.9 -> 158.8 mm, vias 4 -> 23
- net EXP_SCL: track 0.00 -> 82.5 mm, vias 0 -> 12
- net EXP_SDA: track 0.00 -> 75.0 mm, vias 0 -> 10
- net EXP_P7: track 0.00 -> 65.5 mm, vias 0 -> 4
- net FOX_RX: track 0.00 -> 61.6 mm, vias 0 -> 11
- net EXP_P3: track 0.00 -> 58.9 mm, vias 0 -> 4
- net V3V3: track 459.7 -> 514.3 mm, vias 9 -> 15
- net HDR_P7: track 0.00 -> 51.9 mm
- net HDR_P3: track 0.00 -> 50.7 mm, vias 0 -> 1
- net GND: track 1071.5 -> 1119.7 mm, vias 67 -> 108
- net FOX_GND: track 0.00 -> 41.0 mm, vias 0 -> 1
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Other:
- board text added: "ARDF-TX M6-L2"
- board text added: "FOXPRO G/D/V0"
- board text added: "GPIO 3V3 10mA"
- board text added: "LORA ANT"
- board text added: "WIFI 2.4G"
- board text removed: "ARDF-TX L1"
