File: hardware/80m/production/01_source_interface.kicad_sch (KiCad schematic)
At the start: 22 parts, among them J101 IDC16 controller, U101 SI5351A-B-GT, Y101 25 MHz / CL10 pF

Commit message: M4A-V1R1: close RF80 standard-JLCPCB prototype manufacturing candidate
Correct manufacturer-specific component holes for ordinary PTH tolerances, move small artwork to assembly layers, and add native DFM and fit regressions. Preserve RF nets and routing, generate isolated five-board fabrication datasets, and propose the V1R1-first evaluation transition without changing historical approvals. Physical qualification remains NOT_RUN.
Parts:
- J101: Engineering_Note Maker61201621621:27.98mm length,17.78mm span,2.54mm pitch; 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 -> V1R1:1.40mm ordinary finished PTH,1.90mm lands. Maker squar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
