File: hardware/80m/production/05_power.kicad_sch (KiCad schematic)
At the start: 22 parts, among them J301 RAW protected pack, Q301 BSS138BK,215, Q302 BSS138BK,215, U301 TPS54302DDCT, U302 TPS22810DBVR

Commit message: M4A-V1R1: close RF80 standard-JLCPCB prototype manufacturing candidate
Correct manufacturer-specific component holes for ordinary PTH tolerances, move small artwork to assembly layers, and add native DFM and fit regressions. Preserve RF nets and routing, generate isolated five-board fabrication datasets, and propose the V1R1-first evaluation transition without changing historical approvals. Physical qualification remains NOT_RUN.
Parts:
- J301: footprint Connector_JST:JST_VH_B2P-VH_1x02_P3.96mm_Vertical -> ARDF_TX:JST_VH_B2P_StandardPTH; Engineering_Note Pin1 positive,2 power return. Module input must come from e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 -> V1R1:1.90mm ordinary finished PTH. Maker1.14mm square, tole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
