File: hardware/80m/production/08_normal_rf.kicad_sch (KiCad schematic)
At the start: 22 parts, among them Q401 BSS138BK,215, Q402 IRF610PBF-BE3, Q403 BD140 / ST, Q404 DMN2056U-7, Q405 BSS138BK,215, T401 9T + 9T bifilar / FT-50A-43, U401 LM5134BMF/NOPB

Commit message: M4A-V1R1: close RF80 standard-JLCPCB prototype manufacturing candidate
Correct manufacturer-specific component holes for ordinary PTH tolerances, move small artwork to assembly layers, and add native DFM and fit regressions. Preserve RF nets and routing, generate isolated five-board fabrication datasets, and propose the V1R1-first evaluation transition without changing historical approvals. Physical qualification remains NOT_RUN.
Parts:
- Q402: footprint ARDF_TX:TO220_Vertical_1p3Drill -> ARDF_TX:Vishay_IRF610_TO220_StandardPTH; Engineering_Note 200V VDS, +/-20V gate. Tab=drain; electrically insulating s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 -> V1R1:Vishay IRF610PbF-BE3, exact Siliconix92506 drawing.1G/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
- Q403: footprint ARDF_TX:ST_BD140_SOT32_1p3Drill -> ARDF_TX:ST_BD140_SOT32_StandardPTH; Engineering_Note ST BD140, May2008 Rev5 Fig1/p7 drawing0016114E:1BASE,2COLLE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 -> V1R1:ST BD140 SOT32 drawing0016114E,1B/2C/3E;180deg/illustr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
