File: hardware/80m/production/09_normal_filter.kicad_sch (KiCad schematic)
At the start: 11 parts, among them J401 NORMAL 50ohm reference

Commit message: M4A-V1R1: close RF80 standard-JLCPCB prototype manufacturing candidate
Correct manufacturer-specific component holes for ordinary PTH tolerances, move small artwork to assembly layers, and add native DFM and fit regressions. Preserve RF nets and routing, generate isolated five-board fabrication datasets, and propose the V1R1-first evaluation transition without changing historical approvals. Physical qualification remains NOT_RUN.
Parts:
- J401: footprint TerminalBlock_Phoenix:TerminalBlock_Phoenix_MKDS-1-2-3.81_1x02_P3.81mm_Horizontal -> ARDF_TX:Phoenix_1727010_StandardPTH; Engineering_Note Low-cost screw terminal, not controlled50ohm coax. Define t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 -> V1R1:1.30mm ordinary finished PTH. Maker0.5x0.9mm pins; no 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
