File: hardware/80m/production/11_fox_filter.kicad_sch (KiCad schematic)
At the start: 19 parts, among them J502 FOX ONLY / compact

Commit message: M4A-V1R1: close RF80 standard-JLCPCB prototype manufacturing candidate
Correct manufacturer-specific component holes for ordinary PTH tolerances, move small artwork to assembly layers, and add native DFM and fit regressions. Preserve RF nets and routing, generate isolated five-board fabrication datasets, and propose the V1R1-first evaluation transition without changing historical approvals. Physical qualification remains NOT_RUN.
Parts:
- J502: footprint Connector_JST:JST_XH_B3B-XH-A_1x03_P2.50mm_Vertical -> ARDF_TX:JST_XH_B3B_StandardPTH; Engineering_Note Plugshorts3to2. MismatchedwithJ401normalterminalandJ301VH. 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 -> V1R1:1.30mm ordinary finished PTH,1.90x1.95mm lands. Maker0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
