File: hardware/80m/production/RF80_V1.kicad_pcb (KiCad board)
At the start: 2 copper layers, 150 x 110 mm, 217 parts, among them J101 IDC16 controller, J301 RAW protected pack, J401 NORMAL 50ohm reference, J502 FOX ONLY / compact, Q201 BSS138BK,215, Q225 BSS138BK,215, Q226 BSS138BK,215, Q227 BSS138BK,215, Q228 BSS138BK,215, Q229 BSS138BK,215, Q301 BSS138BK,215, Q302 BSS138BK,215, Q401 BSS138BK,215, Q402 IRF610PBF-BE3, Q403 BD140 / ST, Q404 DMN2056U-7, Q405 BSS138BK,215, Q406 BSS138BK,215, Q501 MMBT3906,215, Q502 BSS138BK,215, Q503 MMBT3904,215, Q504 MMBT3904,215, T401 9T + 9T bifilar / FT-50A-43, U101 SI5351A-B-GT, U201 MCP100T-300I/TT, U202 74HC123D,653, U203 74HC14D,653, U211 74HC21D,653, U212 74HC00D,653, U221 74HC11D,653, U222 74HC08D,653, U223 74HC74D,653, U224 74HC174D,653, U301 TPS54302DDCT, U302 TPS22810DBVR, U311 TL431AIDBZR, U312 LM339BIDR, U313 INA180A1IDBVT, U314 LM393BIDR, U401 LM5134BMF/NOPB, U501 SN74AC00DR, Y101 25 MHz / CL10 pF

Commit message: M4A-V1R1: close RF80 standard-JLCPCB prototype manufacturing candidate
Correct manufacturer-specific component holes for ordinary PTH tolerances, move small artwork to assembly layers, and add native DFM and fit regressions. Preserve RF nets and routing, generate isolated five-board fabrication datasets, and propose the V1R1-first evaluation transition without changing historical approvals. Physical qualification remains NOT_RUN.
Parts:
- J301: footprint Connector_JST:JST_VH_B2P-VH_1x02_P3.96mm_Vertical -> ARDF_TX:JST_VH_B2P_StandardPTH
- J401: footprint TerminalBlock_Phoenix:TerminalBlock_Phoenix_MKDS-1-2-3.81_1x02_P3.81mm_Horizontal -> ARDF_TX:Phoenix_1727010_StandardPTH
- J502: footprint Connector_JST:JST_XH_B3B-XH-A_1x03_P2.50mm_Vertical -> ARDF_TX:JST_XH_B3B_StandardPTH
- Q402: footprint ARDF_TX:TO220_Vertical_1p3Drill -> ARDF_TX:Vishay_IRF610_TO220_StandardPTH
- Q403: footprint ARDF_TX:ST_BD140_SOT32_1p3Drill -> ARDF_TX:ST_BD140_SOT32_StandardPTH
Other:
- board text added: "FOX: R228 R348 R349"
- board text added: "FULL:4S FOX:2S"
- board text added: "INSULATE DRAIN TAB"
- board text added: "J101 CTRL 3V3"
- board text added: "J101-1"
- board text added: "J301 1=BAT+ 2=GND"
- board text added: "J301-1"
- board text added: "J401 NORMAL RF"
- board text added: "J401-1"
- board text added: "J502 FOX 10mW"
- board text added: "J502-1"
- board text added: "RF80 V1R1 / EVAL - NOT RELEASED"
- board text added: "TP101"
- board text added: "TP102"
- board text added: "TP513"
- board text added: "TP703"
- board text added: "TP723"
